Commit message: rover listening to topics

File: ros2/scr/lunabotics_description/urdf/basic_rover.urdf (robot description, URDF)
Before this commit: robot basic_rover, 5 links, 4 joints
Joints:
- joint front_left_wheel_joint: axis (none) -> 0 1 0; type fixed -> continuous
- joint front_right_wheel_joint: axis (none) -> 0 1 0; type fixed -> continuous
- joint rear_left_wheel_joint: axis (none) -> 0 1 0; type fixed -> continuous
- joint rear_right_wheel_joint: axis (none) -> 0 1 0; type fixed -> continuous
