Commit message: 2d Lidar for SLAM integration

File: luna_ws/src/luna_sim/description/lidar.xacro (robot description, xacro)
@@ -32,5 +32,5 @@
     <sensor name="lidar_3d" type="gpu_ray">
       <always_on>true</always_on>
-      <visualize>true</visualize>
+      <visualize>false</visualize>
       <update_rate>10</update_rate>
       <ray>

File: luna_ws/src/luna_sim/description/rover.urdf.xacro (robot description, xacro)
@@ -3,4 +3,4 @@
     <xacro:include filename="ros2_control.xacro" />
     <xacro:include filename="depth_camera.xacro" />
-    <xacro:include filename="lidar.xacro" />
+    <xacro:include filename="lidar_2d.xacro" />
 </robot>

File: luna_ws/src/luna_sim/description/rover_core.xacro (robot description, xacro)
@@ -42,4 +42,12 @@
     <material>Gazebo/Grey</material>
   </gazebo>
+    <!-- BASE FOOTPRINT (ground-projected base frame for SLAM/Nav2) -->
+  <joint name="base_footprint_joint" type="fixed">
+    <parent link="base_link"/>
+    <child link="base_footprint"/>
+    <origin xyz="0 0 0" rpy="0 0 0 "/>
+  </joint>
+  <link name="base_footprint">
+  </link>
   <!-- Helper macro for a wheel -->
   <xacro:macro name="wheel_link" params="name">
