Commit message: 3d lidar added

File: qpl_ws/src/qpl_rover/description/lidar.xacro (robot description, xacro)
@@ -1,10 +1,8 @@
 <?xml version="1.0"?>
 <robot xmlns:xacro="http://www.ros.org/wiki/xacro">
-  <!-- Mount lidar to rover -->
   <joint name="lidar_joint" type="fixed">
-    <parent link="base_link"/>
+    <parent link="base_footprint"/>
     <child link="lidar_link"/>
-    <!-- top-center position: adjust as needed -->
-    <origin xyz="0 0 0.3" rpy="0 0 0"/>
+    <origin xyz="0 0 0.30" rpy="0 0 0"/>
   </joint>
   <link name="lidar_link">
@@ -20,5 +18,4 @@
       </geometry>
     </collision>
-    <!-- small inertia so Gazebo is happy -->
     <inertial>
       <origin xyz="0 0 0" rpy="0 0 0"/>
@@ -27,5 +24,4 @@
     </inertial>
   </link>
-  <!-- Gazebo 3D lidar sensor -->
   <gazebo reference="lidar_link">
     <material>Gazebo/Black</material>
@@ -36,5 +32,4 @@
       <ray>
         <scan>
-          <!-- Horizontal scanning (360 degrees) -->
           <horizontal>
             <samples>360</samples>
@@ -43,10 +38,9 @@
             <max_angle>3.14159</max_angle>
           </horizontal>
-          <!-- Vertical scanning (adds 3D capability) -->
           <vertical>
             <samples>16</samples>
             <resolution>1.0</resolution>
-            <min_angle>-0.2617</min_angle>  <!-- -15 degrees -->
-            <max_angle>0.2617</max_angle>   <!-- +15 degrees -->
+            <min_angle>-0.2617</min_angle>
+            <max_angle>0.2617</max_angle>
           </vertical>
         </scan>
@@ -63,9 +57,7 @@
       </ray>
       <plugin name="lidar_3d_controller" filename="libgazebo_ros_ray_sensor.so">
-        <!-- frame published in PointCloud2 header -->
         <frame_name>lidar_link</frame_name>
-        <!-- topic name for PointCloud2 messages -->
         <output_type>sensor_msgs/PointCloud2</output_type>
-        <topic_name>points</topic_name>
+        <topic_name>/points</topic_name>
       </plugin>
     </sensor>

Commit message: nav2 params file

File: qpl_ws/src/qpl_rover/description/lidar.xacro (robot description, xacro)
@@ -1,10 +1,10 @@
 <?xml version="1.0"?>
 <robot xmlns:xacro="http://www.ros.org/wiki/xacro">
-  <joint name="lidar_joint" type="fixed">
+  <joint name="laser_joint" type="fixed">
     <parent link="base_footprint"/>
-    <child link="lidar_link"/>
+    <child link="laser_frame"/>
     <origin xyz="0 0 0.30" rpy="0 0 0"/>
   </joint>
-  <link name="lidar_link">
+  <link name="laser_frame">
     <visual>
       <geometry>
@@ -18,34 +18,32 @@
       </geometry>
     </collision>
-    <inertial>
+    <xacro:inertial_cylinder mass="0.1" length="0.04" radius="0.05">
       <origin xyz="0 0 0" rpy="0 0 0"/>
-      <mass value="0.125"/>
-      <inertia ixx="1e-4" ixy="0" ixz="0" iyy="1e-4" iyz="0" izz="1e-4"/>
-    </inertial>
+    </xacro:inertial_cylinder>
   </link>
-  <gazebo reference="lidar_link">
+  <gazebo reference="laser_frame">
     <material>Gazebo/Black</material>
-    <sensor name="lidar_3d" type="gpu_ray">
-      <always_on>true</always_on>
+    <sensor name="laser_3d" type="gpu_ray">
+      <pose>0 0 0 0 0 0</pose>
       <visualize>false</visualize>
-      <update_rate>10</update_rate>
+      <update_rate>15</update_rate>
       <ray>
         <scan>
           <horizontal>
-            <samples>360</samples>
-            <resolution>1.0</resolution>
+            <samples>180</samples>
+            <resolution>1</resolution>
             <min_angle>-3.14159</min_angle>
             <max_angle>3.14159</max_angle>
           </horizontal>
           <vertical>
-            <samples>16</samples>
-            <resolution>1.0</resolution>
-            <min_angle>-0.2617</min_angle>
-            <max_angle>0.2617</max_angle>
+            <samples>8</samples>
+            <resolution>1</resolution>
+            <min_angle>-0.261799</min_angle>
+            <max_angle>0.261799</max_angle>
           </vertical>
         </scan>
         <range>
-          <min>0.15</min>
-          <max>20.0</max>
+          <min>0.30</min>
+          <max>12.0</max>
           <resolution>0.01</resolution>
         </range>
@@ -56,8 +54,10 @@
         </noise>
       </ray>
-      <plugin name="lidar_3d_controller" filename="libgazebo_ros_ray_sensor.so">
-        <frame_name>lidar_link</frame_name>
+      <plugin name="laser_controller" filename="libgazebo_ros_ray_sensor.so">
+        <ros>
+          <argument>~/out:=/points</argument>
+        </ros>
         <output_type>sensor_msgs/PointCloud2</output_type>
-        <topic_name>/points</topic_name>
+        <frame_name>laser_frame</frame_name>
       </plugin>
     </sensor>

File: qpl_ws/src/qpl_rover/description/rover_core.xacro (robot description, xacro)
@@ -68,5 +68,5 @@
       <!-- skid-steer turning: reduce lateral friction -->
       <mu1>1.4</mu1>
-      <mu2>0.07</mu2>
+      <mu2>0.1</mu2>
       <!-- optional: allow lateral slip -->
       <slip1>0.0</slip1>
