Commit message: Changed depth camera to use best effort

File: qpl_ws/src/qpl_rover/description/depth_camera.xacro (robot description, xacro)
@@ -1,68 +1,79 @@
 <?xml version="1.0"?>
 <robot xmlns:xacro="http://www.ros.org/wiki/xacro">
-  <!-- Mount camera to rover -->
-  <joint name="camera_joint" type="fixed">
-    <parent link="base_link"/>
-    <child link="camera_link"/>
-    <!-- front-top-ish: adjust as needed -->
-    <origin xyz="0.25 0 0.15" rpy="0 0 0"/>
-  </joint>
-  <link name="camera_link">
-    <visual>
-      <geometry>
-        <box size="0.010 0.03 0.03"/>
-      </geometry>
-      <material name="red"/>
-    </visual>
-    <collision>
-      <geometry>
-        <box size="0.010 0.03 0.03"/>
-      </geometry>
-    </collision>
-    <!-- small inertia so Gazebo is happy -->
-    <inertial>
-      <origin xyz="0 0 0" rpy="0 0 0"/>
-      <mass value="0.05"/>
-      <inertia ixx="1e-5" ixy="0" ixz="0" iyy="1e-5" iyz="0" izz="1e-5"/>
-    </inertial>
-  </link>
-  <!-- Optical frame (REP-103/REP-105 style) -->
-  <joint name="camera_optical_joint" type="fixed">
-    <parent link="camera_link"/>
-    <child link="camera_link_optical"/>
-    <origin xyz="0 0 0" rpy="${-pi/2} 0 ${-pi/2}"/>
-  </joint>
-  <link name="camera_link_optical"/>
-  <!-- Gazebo depth sensor -->
-  <gazebo reference="camera_link">
-    <material>Gazebo/Red</material>
-    <sensor name="depth_camera" type="depth">
-      <always_on>true</always_on>
-      <visualize>true</visualize>
-      <update_rate>10</update_rate>
-      <camera>
-        <horizontal_fov>1.089</horizontal_fov>
-        <image>
-          <format>B8G8R8</format>
-          <width>640</width>
-          <height>480</height>
-        </image>
-        <clip>
-          <near>0.05</near>
-          <far>8.0</far>
-        </clip>
-      </camera>
-      <plugin name="depth_camera_controller" filename="libgazebo_ros_camera.so">
-        <!-- frame published in CameraInfo -->
-        <frame_name>camera_link_optical</frame_name>
-        <!-- predictable topic names -->
-        <camera_name>depth_camera</camera_name>
-        <image_topic_name>rgb/image_raw</image_topic_name>
-        <camera_info_topic_name>rgb/camera_info</camera_info_topic_name>
-        <depth_image_topic_name>depth/image_raw</depth_image_topic_name>
-        <depth_camera_info_topic_name>depth/camera_info</depth_camera_info_topic_name>
-        <point_cloud_topic_name>depth/points</point_cloud_topic_name>
-      </plugin>
-    </sensor>
-  </gazebo>
+    <!-- Mount camera to rover -->
+    <joint name="camera_joint" type="fixed">
+        <parent link="base_link"/>
+        <child link="camera_link"/>
+        <!-- front-top-ish: adjust as needed -->
+        <origin xyz="0.25 0 0.15" rpy="0 0 0"/>
+    </joint>
+    <link name="camera_link">
+        <visual>
+            <geometry>
+                <box size="0.010 0.03 0.03"/>
+            </geometry>
+            <material name="red"/>
+        </visual>
+        <collision>
+            <geometry>
+                <box size="0.010 0.03 0.03"/>
+            </geometry>
+        </collision>
+        <!-- small inertia so Gazebo is happy -->
+        <inertial>
+            <origin xyz="0 0 0" rpy="0 0 0"/>
+            <mass value="0.05"/>
+            <inertia ixx="1e-5" ixy="0" ixz="0" iyy="1e-5" iyz="0" izz="1e-5"/>
+        </inertial>
+    </link>
+    <!-- Optical frame (REP-103/REP-105 style) -->
+    <joint name="camera_optical_joint" type="fixed">
+        <parent link="camera_link"/>
+        <child link="camera_link_optical"/>
+        <origin xyz="0 0 0" rpy="${-pi/2} 0 ${-pi/2}"/>
+    </joint>
+    <link name="camera_link_optical"/>
+    <!-- Gazebo depth sensor -->
+    <gazebo reference="camera_link">
+        <material>Gazebo/Red</material>
+        <sensor name="depth_camera" type="depth">
+            <always_on>true</always_on>
+            <visualize>true</visualize>
+            <update_rate>10</update_rate>
+            <camera>
+                <horizontal_fov>1.089</horizontal_fov>
+                <image>
+                    <format>B8G8R8</format>
+                    <width>640</width>
+                    <height>480</height>
+                </image>
+                <clip>
+                    <near>0.05</near>
+                    <far>8.0</far>
+                </clip>
+            </camera>
+            <plugin name="depth_camera_controller" filename="libgazebo_ros_camera.so">
+                <!-- frame published in CameraInfo -->
+                <frame_name>camera_link_optical</frame_name>
+                <!-- predictable topic names -->
+                <camera_name>depth_camera</camera_name>
+                <image_topic_name>rgb/image_raw</image_topic_name>
+                <camera_info_topic_name>rgb/camera_info</camera_info_topic_name>
+                <depth_image_topic_name>depth/image_raw</depth_image_topic_name>
+                <depth_camera_info_topic_name>depth/camera_info</depth_camera_info_topic_name>
+                <point_cloud_topic_name>depth/points</point_cloud_topic_name>
+                <ros>
+                    <qos>
+                        <topic name="/depth_camera/image_raw">
+                            <publisher>
+                                <reliability>best_effort</reliability>
+                                <durability>volatile</durability>
+                                <history depth="1">keep_last</history>
+                            </publisher>
+                        </topic>
+                    </qos>
+                </ros>
+            </plugin>
+        </sensor>
+    </gazebo>
 </robot>

Commit message: Reverted accidental indent changes

File: qpl_ws/src/qpl_rover/description/depth_camera.xacro (robot description, xacro)
@@ -1,79 +1,68 @@
 <?xml version="1.0"?>
 <robot xmlns:xacro="http://www.ros.org/wiki/xacro">
-    <!-- Mount camera to rover -->
-    <joint name="camera_joint" type="fixed">
-        <parent link="base_link"/>
-        <child link="camera_link"/>
-        <!-- front-top-ish: adjust as needed -->
-        <origin xyz="0.25 0 0.15" rpy="0 0 0"/>
-    </joint>
-    <link name="camera_link">
-        <visual>
-            <geometry>
-                <box size="0.010 0.03 0.03"/>
-            </geometry>
-            <material name="red"/>
-        </visual>
-        <collision>
-            <geometry>
-                <box size="0.010 0.03 0.03"/>
-            </geometry>
-        </collision>
-        <!-- small inertia so Gazebo is happy -->
-        <inertial>
-            <origin xyz="0 0 0" rpy="0 0 0"/>
-            <mass value="0.05"/>
-            <inertia ixx="1e-5" ixy="0" ixz="0" iyy="1e-5" iyz="0" izz="1e-5"/>
-        </inertial>
-    </link>
-    <!-- Optical frame (REP-103/REP-105 style) -->
-    <joint name="camera_optical_joint" type="fixed">
-        <parent link="camera_link"/>
-        <child link="camera_link_optical"/>
-        <origin xyz="0 0 0" rpy="${-pi/2} 0 ${-pi/2}"/>
-    </joint>
-    <link name="camera_link_optical"/>
-    <!-- Gazebo depth sensor -->
-    <gazebo reference="camera_link">
-        <material>Gazebo/Red</material>
-        <sensor name="depth_camera" type="depth">
-            <always_on>true</always_on>
-            <visualize>true</visualize>
-            <update_rate>10</update_rate>
-            <camera>
-                <horizontal_fov>1.089</horizontal_fov>
-                <image>
-                    <format>B8G8R8</format>
-                    <width>640</width>
-                    <height>480</height>
-                </image>
-                <clip>
-                    <near>0.05</near>
-                    <far>8.0</far>
-                </clip>
-            </camera>
-            <plugin name="depth_camera_controller" filename="libgazebo_ros_camera.so">
-                <!-- frame published in CameraInfo -->
-                <frame_name>camera_link_optical</frame_name>
-                <!-- predictable topic names -->
-                <camera_name>depth_camera</camera_name>
-                <image_topic_name>rgb/image_raw</image_topic_name>
-                <camera_info_topic_name>rgb/camera_info</camera_info_topic_name>
-                <depth_image_topic_name>depth/image_raw</depth_image_topic_name>
-                <depth_camera_info_topic_name>depth/camera_info</depth_camera_info_topic_name>
-                <point_cloud_topic_name>depth/points</point_cloud_topic_name>
-                <ros>
-                    <qos>
-                        <topic name="/depth_camera/image_raw">
-                            <publisher>
-                                <reliability>best_effort</reliability>
-                                <durability>volatile</durability>
-                                <history depth="1">keep_last</history>
-                            </publisher>
-                        </topic>
-                    </qos>
-                </ros>
-            </plugin>
-        </sensor>
-    </gazebo>
+  <!-- Mount camera to rover -->
+  <joint name="camera_joint" type="fixed">
+    <parent link="base_link"/>
+    <child link="camera_link"/>
+    <!-- front-top-ish: adjust as needed -->
+    <origin xyz="0.25 0 0.15" rpy="0 0 0"/>
+  </joint>
+  <link name="camera_link">
+    <visual>
+      <geometry>
+        <box size="0.010 0.03 0.03"/>
+      </geometry>
+      <material name="red"/>
+    </visual>
+    <collision>
+      <geometry>
+        <box size="0.010 0.03 0.03"/>
+      </geometry>
+    </collision>
+    <!-- small inertia so Gazebo is happy -->
+    <inertial>
+      <origin xyz="0 0 0" rpy="0 0 0"/>
+      <mass value="0.05"/>
+      <inertia ixx="1e-5" ixy="0" ixz="0" iyy="1e-5" iyz="0" izz="1e-5"/>
+    </inertial>
+  </link>
+  <!-- Optical frame (REP-103/REP-105 style) -->
+  <joint name="camera_optical_joint" type="fixed">
+    <parent link="camera_link"/>
+    <child link="camera_link_optical"/>
+    <origin xyz="0 0 0" rpy="${-pi/2} 0 ${-pi/2}"/>
+  </joint>
+  <link name="camera_link_optical"/>
+  <!-- Gazebo depth sensor -->
+  <gazebo reference="camera_link">
+    <material>Gazebo/Red</material>
+    <sensor name="depth_camera" type="depth">
+      <always_on>true</always_on>
+      <visualize>true</visualize>
+      <update_rate>10</update_rate>
+      <camera>
+        <horizontal_fov>1.089</horizontal_fov>
+        <image>
+          <format>B8G8R8</format>
+          <width>640</width>
+          <height>480</height>
+        </image>
+        <clip>
+          <near>0.05</near>
+          <far>8.0</far>
+        </clip>
+      </camera>
+      <plugin name="depth_camera_controller" filename="libgazebo_ros_camera.so">
+        <!-- frame published in CameraInfo -->
+        <frame_name>camera_link_optical</frame_name>
+        <!-- predictable topic names -->
+        <camera_name>depth_camera</camera_name>
+        <image_topic_name>rgb/image_raw</image_topic_name>
+        <camera_info_topic_name>rgb/camera_info</camera_info_topic_name>
+        <depth_image_topic_name>depth/image_raw</depth_image_topic_name>
+        <depth_camera_info_topic_name>depth/camera_info</depth_camera_info_topic_name>
+        <point_cloud_topic_name>depth/points</point_cloud_topic_name>
+      </plugin>
+    </sensor>
+  </gazebo>
 </robot>
