Commit message: fixed imu fusion

File: qpl_ws/src/qpl_rover/description/imu.xacro (robot description, xacro)
@@ -5,4 +5,5 @@
     <link name="imu_link">
       <inertial>
+        <origin xyz="0 0 0" rpy="0 0 0"/>
         <mass value="0.01"/>
         <inertia ixx="1e-6" iyy="1e-6" izz="1e-6"
@@ -13,5 +14,4 @@
       <parent link="${parent_link}"/>
       <child link="imu_link"/>
-      <!-- Position on robot (tweak if needed) -->
       <origin xyz="0 0 0.15" rpy="0 0 0"/>
     </joint>
@@ -21,4 +21,5 @@
         <update_rate>50</update_rate>
         <visualize>false</visualize>
+        <topic>imu</topic>
         <imu>
           <angular_velocity>
@@ -27,4 +28,6 @@
                 <mean>0.0</mean>
                 <stddev>0.0002</stddev>
+                <bias_mean>0.0000075</bias_mean>
+                <bias_stddev>0.0000008</bias_stddev>
               </noise>
             </x>
@@ -33,4 +36,6 @@
                 <mean>0.0</mean>
                 <stddev>0.0002</stddev>
+                <bias_mean>0.0000075</bias_mean>
+                <bias_stddev>0.0000008</bias_stddev>
               </noise>
             </y>
@@ -39,7 +44,35 @@
                 <mean>0.0</mean>
                 <stddev>0.0002</stddev>
+                <bias_mean>0.0000075</bias_mean>
+                <bias_stddev>0.0000008</bias_stddev>
               </noise>
             </z>
           </angular_velocity>
+          <linear_acceleration>
+            <x>
+              <noise type="gaussian">
+                <mean>0.0</mean>
+                <stddev>0.017</stddev>
+                <bias_mean>0.1</bias_mean>
+                <bias_stddev>0.001</bias_stddev>
+              </noise>
+            </x>
+            <y>
+              <noise type="gaussian">
+                <mean>0.0</mean>
+                <stddev>0.017</stddev>
+                <bias_mean>0.1</bias_mean>
+                <bias_stddev>0.001</bias_stddev>
+              </noise>
+            </y>
+            <z>
+              <noise type="gaussian">
+                <mean>0.0</mean>
+                <stddev>0.017</stddev>
+                <bias_mean>0.1</bias_mean>
+                <bias_stddev>0.001</bias_stddev>
+              </noise>
+            </z>
+          </linear_acceleration>
         </imu>
         <plugin name="imu_plugin" filename="libgazebo_ros_imu_sensor.so">
@@ -48,7 +81,9 @@
           </ros>
           <frame_name>imu_link</frame_name>
+          <initial_orientation_as_reference>false</initial_orientation_as_reference>
         </plugin>
       </sensor>
     </gazebo>
   </xacro:macro>
+  <xacro:imu_sensor parent_link="base_link"/>
 </robot>

File: qpl_ws/src/qpl_rover/description/rover.urdf.xacro (robot description, xacro)
@@ -7,4 +7,5 @@
         <xacro:include filename="ros2_control.xacro" />
     </xacro:if>
+    <xacro:include filename="imu.xacro" />
     <xacro:include filename="depth_camera.xacro" />
     <xacro:include filename="back_camera.xacro" />

File: qpl_ws/src/qpl_rover/description/rover_core.xacro (robot description, xacro)
@@ -9,5 +9,5 @@
   <xacro:property name="base_y" value="0.30"/>
   <xacro:property name="base_z" value="0.18"/>
-  <xacro:property name="wheel_r" value="0.08"/>
+  <xacro:property name="wheel_r" value="0.10"/>
   <!-- base_link is located above the ground by wheel radius + half the base height -->
   <xacro:property name="base_z_origin" value="${wheel_r + base_z/2}"/>
@@ -68,5 +68,5 @@
       <!-- skid-steer turning: reduce lateral friction -->
       <mu1>1.4</mu1>
-      <mu2>0.1</mu2>
+      <mu2>0.2</mu2>
       <!-- optional: allow lateral slip -->
       <slip1>0.0</slip1>
