Commit message: fixed slam

File: qpl_ws/src/qpl_rover/description/back_camera.xacro (robot description, xacro)
@@ -1,17 +1,12 @@
+<?xml version="1.0"?>
 <robot xmlns:xacro="http://www.ros.org/wiki/xacro">
-  <!-- IMX219 Camera Module 120 FOV - Back Camera -->
-  <!-- This camera simulates the IMX219 sensor with wide angle lens -->
-  <!-- Mount camera to rover -->
   <joint name="back_camera_joint" type="fixed">
     <parent link="base_link"/>
     <child link="back_camera_link"/>
-    <!-- Position: back-center-top of rover, facing backward -->
     <origin xyz="-0.25 0 0.18" rpy="0 0 ${pi}"/>
   </joint>
-  <!-- Camera link (physical body) -->
   <link name="back_camera_link">
     <visual>
       <geometry>
-        <!-- IMX219 module is roughly 25mm x 24mm x 9mm -->
         <box size="0.025 0.024 0.009"/>
       </geometry>
@@ -23,14 +18,10 @@
       </geometry>
     </collision>
-    <!-- Light inertia for small camera module -->
     <inertial>
       <origin xyz="0 0 0" rpy="0 0 0"/>
-      <mass value="0.003"/>  <!-- ~3 grams -->
+      <mass value="0.003"/>
       <inertia ixx="1e-6" ixy="0" ixz="0" iyy="1e-6" iyz="0" izz="1e-6"/>
     </inertial>
   </link>
-  <!-- Optical frame (REP-103/REP-105 convention) -->
-  <!-- This transforms from camera_link to optical frame: -->
-  <!-- X-right, Y-down, Z-forward (optical convention) -->
   <joint name="back_camera_optical_joint" type="fixed">
     <parent link="back_camera_link"/>
@@ -39,5 +30,4 @@
   </joint>
   <link name="back_camera_link_optical"/>
-  <!-- Gazebo camera sensor plugin -->
   <gazebo reference="back_camera_link">
     <material>Gazebo/Blue</material>
@@ -45,29 +35,24 @@
       <always_on>true</always_on>
       <visualize>true</visualize>
-      <update_rate>30</update_rate>  <!-- IMX219 can do up to 30 fps at full resolution -->
+      <update_rate>30</update_rate>
       <camera>
-        <!-- 120 degrees horizontal FOV = 2.094 radians -->
         <horizontal_fov>2.0944</horizontal_fov>
         <image>
-          <!-- IMX219 native resolution is 3280x2464, but using common operational resolution -->
           <format>R8G8B8</format>
-          <width>1920</width>   <!-- 1080p resolution (common for robotics) -->
+          <width>1920</width>
           <height>1080</height>
         </image>
         <clip>
-          <near>0.02</near>  <!-- 2cm minimum distance -->
-          <far>300</far>     <!-- 300m maximum distance (effectively infinite for this camera) -->
+          <near>0.02</near>
+          <far>300</far>
         </clip>
-        <!-- Noise model for more realistic simulation -->
         <noise>
           <type>gaussian</type>
           <mean>0.0</mean>
-          <stddev>0.007</stddev>  <!-- Small amount of noise -->
+          <stddev>0.007</stddev>
         </noise>
       </camera>
       <plugin name="back_camera_controller" filename="libgazebo_ros_camera.so">
-        <!-- Frame name for TF and CameraInfo -->
         <frame_name>back_camera_link_optical</frame_name>
-        <!-- ROS 2 remapping -->
         <ros>
           <namespace>/</namespace>
@@ -75,5 +60,4 @@
           <remapping>camera_info:=back_camera/camera_info</remapping>
         </ros>
-        <!-- Distortion parameters (can be adjusted for lens characteristics) -->
         <distortion_k1>0.0</distortion_k1>
         <distortion_k2>0.0</distortion_k2>
@@ -81,5 +65,4 @@
         <distortion_t1>0.0</distortion_t1>
         <distortion_t2>0.0</distortion_t2>
-        <!-- CameraInfo manager settings -->
         <hack_baseline>0.0</hack_baseline>
       </plugin>

File: qpl_ws/src/qpl_rover/description/depth_camera.xacro (robot description, xacro)
@@ -1,2 +1,3 @@
+<?xml version="1.0"?>
 <robot xmlns:xacro="http://www.ros.org/wiki/xacro">
   <!-- Mount camera to rover -->

File: qpl_ws/src/qpl_rover/description/inertial_macros.xacro (robot description, xacro)
@@ -1,11 +1,4 @@
-<robot xmlns:xacro="http://www.ros.org/wiki/xacro" name="inertial_macros">
-  <!--
-    Standard inertial calculations
-    https://en.wikipedia.org/wiki/List_of_moments_of_inertia
-    Notes:
-    - Inertias are expressed about the link frame.
-    - We keep the original macro names for compatibility.
-  -->
-  <!-- Sphere inertia -->
+<?xml version="1.0"?>
+<robot xmlns:xacro="http://www.ros.org/wiki/xacro">
   <xacro:macro name="inertial_sphere" params="mass radius *origin">
     <inertial>
@@ -18,5 +11,4 @@
     </inertial>
   </xacro:macro>
-  <!-- Box inertia (about link frame axes) -->
   <xacro:macro name="inertial_box" params="mass x y z *origin">
     <inertial>
@@ -29,5 +21,4 @@
     </inertial>
   </xacro:macro>
-  <!-- Cylinder inertia (assumes cylinder axis aligned with link Z axis) -->
   <xacro:macro name="inertial_cylinder" params="mass length radius *origin">
     <inertial>
@@ -40,15 +31,8 @@
     </inertial>
   </xacro:macro>
-  <!--
-    Cylinder inertia with axis along link Y.
-    Useful if you decide to align your wheel link frame such that the wheel axle is Y.
-    This just permutes principal moments so the "axis" moment sits on Iyy.
-  -->
   <xacro:macro name="inertial_cylinder_y" params="mass length radius *origin">
     <inertial>
       <xacro:insert_block name="origin"/>
       <mass value="${mass}" />
-      <!-- For a cylinder, inertia about its axis is (1/2) m r^2.
-           If axis is Y, then Iyy is the axial inertia. -->
       <inertia
         ixx="${(1.0/12.0) * mass * (3*radius*radius + length*length)}" ixy="0.0" ixz="0.0"

File: qpl_ws/src/qpl_rover/description/ros2_control.xacro (robot description, xacro)
@@ -1,53 +1,47 @@
+<?xml version="1.0"?>
 <robot xmlns:xacro="http://www.ros.org/wiki/xacro">
-  <!--
-    ros2_control + Gazebo
-    This replaces the old gazebo_ros_diff_drive + gazebo_ros_joint_state_publisher plugins.
-    Gazebo will expose the wheel joints through ros2_control, and we'll run:
-      - joint_state_broadcaster  (publishes /joint_states)
-      - diff_drive_controller    (subscribes to /cmd_vel, publishes /odom + TF)
-  -->
-  <!-- 1) ros2_control hardware definition (GazeboSystem) -->
-    <!-- ros2_control + Gazebo -->
-  <ros2_control name="GazeboSystem" type="system">
-    <hardware>
-      <plugin>gazebo_ros2_control/GazeboSystem</plugin>
-    </hardware>
-    <joint name="front_left_wheel_joint">
-      <command_interface name="velocity">
-          <param name="min_velocity">-10</param>
-          <param name="max_velocity">10</param>
-      </command_interface>
-      <state_interface name="position"/>
-      <state_interface name="velocity"/>
-    </joint>
-    <joint name="front_right_wheel_joint">
-      <command_interface name="velocity">
-          <param name="min_velocity">-10</param>
-          <param name="max_velocity">10</param>
-      </command_interface>
-      <state_interface name="position"/>
-      <state_interface name="velocity"/>
-    </joint>
-    <joint name="rear_left_wheel_joint">
-      <command_interface name="velocity">
+  <xacro:if value="$(arg sim_mode)">
+    <ros2_control name="GazeboSystem" type="system">
+      <hardware>
+        <plugin>gazebo_ros2_control/GazeboSystem</plugin>
+      </hardware>
+      <joint name="front_left_wheel_joint">
+        <command_interface name="velocity">
             <param name="min_velocity">-10</param>
             <param name="max_velocity">10</param>
-      </command_interface>
-      <state_interface name="position"/>
-      <state_interface name="velocity"/>
-    </joint>
-    <joint name="rear_right_wheel_joint">
-      <command_interface name="velocity">
+        </command_interface>
+        <state_interface name="position"/>
+        <state_interface name="velocity"/>
+      </joint>
+      <joint name="front_right_wheel_joint">
+        <command_interface name="velocity">
             <param name="min_velocity">-10</param>
             <param name="max_velocity">10</param>
-      </command_interface>
-      <state_interface name="position"/>
-      <state_interface name="velocity"/>
-    </joint>
-  </ros2_control>
-  <!-- Gazebo plugin that hosts controller_manager -->
+        </command_interface>
+        <state_interface name="position"/>
+        <state_interface name="velocity"/>
+      </joint>
+      <joint name="rear_left_wheel_joint">
+        <command_interface name="velocity">
+              <param name="min_velocity">-10</param>
+              <param name="max_velocity">10</param>
+        </command_interface>
+        <state_interface name="position"/>
+        <state_interface name="velocity"/>
+      </joint>
+      <joint name="rear_right_wheel_joint">
+        <command_interface name="velocity">
+              <param name="min_velocity">-10</param>
+              <param name="max_velocity">10</param>
+        </command_interface>
+        <state_interface name="position"/>
+        <state_interface name="velocity"/>
+      </joint>
+    </ros2_control>
+  </xacro:if>
   <gazebo>
-    <plugin  name="gazebo_ros2_control "  filename="libgazebo_ros2_control.so">
+    <plugin  name="gazebo_ros2_control"  filename="libgazebo_ros2_control.so">
       <parameters>$(find qpl_rover)/config/my_controllers.yaml</parameters>
+      <parameters>$(find qpl_rover)/config/gaz_ros2_ctl_use_sim.yaml</parameters>
     </plugin>
   </gazebo>

File: qpl_ws/src/qpl_rover/description/rover.urdf.xacro (robot description, xacro)
@@ -1,9 +1,12 @@
+<?xml version="1.0"?>
 <robot xmlns:xacro="http://www.ros.org/wiki/xacro"  name="robot">
+    <xacro:arg name="use_ros2_control" default="true"/>
+    <xacro:arg name="sim_mode" default="true"/>
     <xacro:include filename="rover_core.xacro" />
-    <xacro:include filename="ros2_control.xacro" />
+    <xacro:if value="$(arg use_ros2_control)">
+        <xacro:include filename="ros2_control.xacro" />
+    </xacro:if>
     <xacro:include filename="depth_camera.xacro" />
     <xacro:include filename="lidar_2d.xacro" />
     <xacro:include filename="back_camera.xacro" />
-    <xacro:include filename="imu.xacro"/>
-    <xacro:imu_sensor parent_link="base_link"/>
 </robot>

File: qpl_ws/src/qpl_rover/description/rover_core.xacro (robot description, xacro)
@@ -1,38 +1,29 @@
-<robot xmlns:xacro="http://www.ros.org/wiki/xacro" name="robot">
+<?xml version="1.0"?>
+<robot xmlns:xacro="http://www.ros.org/wiki/xacro">
   <xacro:include filename="inertial_macros.xacro"/>
-  <!-- Materials -->
   <material name="gray"><color rgba="0.6 0.6 0.6 1.0"/></material>
   <material name="black"><color rgba="0.05 0.05 0.05 1.0"/></material>
   <material name="red"><color rgba="0.8 0.1 0.1 1.0"/></material>
   <material name="blue"><color rgba="0.2 0.2 1.0 1.0"/></material>
-  <!-- Dimensions (easy to tweak) -->
   <xacro:property name="base_x" value="0.50"/>
   <xacro:property name="base_y" value="0.30"/>
   <xacro:property name="base_z" value="0.18"/>
-  <xacro:property name="base_z_origin" value="0.12"/>
-  <xacro:property name="wheel_r" value="0.10"/>
+    <xacro:property name="wheel_r" value="0.08"/>
+  <xacro:property name="base_z_origin" value="${wheel_r + base_z/2}"/>
   <xacro:property name="wheel_w" value="0.03"/>
-  <!-- Wheel placement (relative to base_link origin) -->
   <xacro:property name="wheel_x_front" value="0.18"/>
   <xacro:property name="wheel_x_rear"  value="-0.18"/>
   <xacro:property name="wheel_y" value="${base_y/2 + wheel_w/2}"/>
-  <!-- Put wheel centers slightly below base collision bottom (base bottom is z=0.0) -->
-  <xacro:property name="wheel_z" value="0.02"/>
-  <!-- BASE LINK (chassis) -->
+  <xacro:property name="wheel_z" value="${wheel_r}"/>
   <link name="base_link">
     <visual>
       <origin xyz="0 0 ${base_z_origin}" rpy="0 0 0"/>
-      <geometry>
-        <box size="${base_x} ${base_y} ${base_z}"/>
-      </geometry>
+      <geometry><box size="${base_x} ${base_y} ${base_z}"/></geometry>
       <material name="gray"/>
     </visual>
     <collision>
       <origin xyz="0 0 ${base_z_origin}" rpy="0 0 0"/>
-      <geometry>
-        <box size="${base_x} ${base_y} ${base_z}"/>
-      </geometry>
+      <geometry><box size="${base_x} ${base_y} ${base_z}"/></geometry>
     </collision>
-    <!-- Use your macro for inertia -->
     <xacro:inertial_box mass="10.0" x="${base_x}" y="${base_y}" z="${base_z}">
       <origin xyz="0 0 ${base_z/2}" rpy="0 0 0"/>
@@ -42,28 +33,22 @@
     <material>Gazebo/Grey</material>
   </gazebo>
-    <!-- BASE FOOTPRINT (ground-projected base frame for SLAM/Nav2) -->
   <joint name="base_footprint_joint" type="fixed">
     <parent link="base_link"/>
     <child link="base_footprint"/>
-    <origin xyz="0 0 0" rpy="0 0 0 "/>
+    <origin xyz="0 0 0" rpy="0 0 0"/>
   </joint>
-  <link name="base_footprint">
-  </link>
-  <!-- Helper macro for a wheel -->
+  <link name="base_footprint"/>
+  <!-- WHEELS -->
   <xacro:macro name="wheel_link" params="name">
     <link name="${name}">
       <visual>
-        <!-- Rotate cylinder so it spins about Y (axle along Y) -->
         <origin xyz="0 0 0" rpy="${pi/2} 0 0"/>
-        <geometry>
-          <cylinder radius="${wheel_r}" length="${wheel_w}"/>
-        </geometry>
+        <geometry><cylinder radius="${wheel_r}" length="${wheel_w}"/></geometry>
         <material name="red"/>
       </visual>
+      <!-- slightly smaller collision helps avoid micro-binding -->
       <collision>
         <origin xyz="0 0 0" rpy="${pi/2} 0 0"/>
-        <geometry>
-          <cylinder radius="${wheel_r}" length="${wheel_w}"/>
-        </geometry>
+        <geometry><cylinder radius="${wheel_r*0.98}" length="${wheel_w*0.95}"/></geometry>
       </collision>
       <xacro:inertial_cylinder mass="0.5" length="${wheel_w}" radius="${wheel_r}">
@@ -71,15 +56,20 @@
       </xacro:inertial_cylinder>
     </link>
+    <!-- ONE gazebo block per wheel -->
     <gazebo reference="${name}">
       <material>Gazebo/Red</material>
+      <fdir1>1 0 0</fdir1>
+      <!-- skid-steer turning: reduce lateral friction -->
+      <mu1>1.0</mu1>
+      <mu2>0.1</mu2>
+      <!-- optional: allow lateral slip -->
+      <slip1>0.0</slip1>
+      <slip2>0.0</slip2>
     </gazebo>
   </xacro:macro>
-  <!-- Create 4 wheels -->
   <xacro:wheel_link name="front_left_wheel"/>
   <xacro:wheel_link name="front_right_wheel"/>
   <xacro:wheel_link name="rear_left_wheel"/>
   <xacro:wheel_link name="rear_right_wheel"/>
-  <!-- Joints -->
-  <!-- NOTE: Axis set to Y so wheel rotates correctly with the visual rotation above -->
   <joint name="front_left_wheel_joint" type="continuous">
     <parent link="base_link"/>
@@ -106,16 +96,3 @@
     <axis xyz="0 1 0"/>
   </joint>
-  <!-- Make REAR wheels (passive) very low friction so they don't fight the driven front wheels -->
-  <gazebo reference="rear_left_wheel">
-    <mu1 value="0.0001"/>
-    <mu2 value="0.0001"/>
-    <slip1 value="1.0"/>
-    <slip2 value="1.0"/>
-  </gazebo>
-  <gazebo reference="rear_right_wheel">
-    <mu1 value="0.0001"/>
-    <mu2 value="0.0001"/>
-    <slip1 value="1.0"/>
-    <slip2 value="1.0"/>
-  </gazebo>
 </robot>

Commit message: Fix AprilTag and back camera parameters to get accurate tf

File: qpl_ws/src/qpl_rover/description/back_camera.xacro (robot description, xacro)
@@ -4,5 +4,5 @@
     <parent link="base_link"/>
     <child link="back_camera_link"/>
-    <origin xyz="-0.25 0 0.18" rpy="0 0 ${pi}"/>
+    <origin xyz="-0.25 0 0.18" rpy="0 0 0"/>
   </joint>
   <link name="back_camera_link">

Commit message: Fixes to get accurate x, y, and yaw values

File: qpl_ws/src/qpl_rover/description/back_camera.xacro (robot description, xacro)
@@ -4,5 +4,5 @@
     <parent link="base_link"/>
     <child link="back_camera_link"/>
-    <origin xyz="-0.25 0 0.18" rpy="0 0 0"/>
+    <origin xyz="-0.25 0 0.18" rpy="0 0 ${pi}"/>
   </joint>
   <link name="back_camera_link">
