Commit message: rear depth cam added

File: qpl_ws/src/qpl_rover/description/depth_camera_front.xacro (robot description, xacro)
@@ -2,11 +2,11 @@
 <robot xmlns:xacro="http://www.ros.org/wiki/xacro">
   <!-- Mount camera to rover -->
-  <joint name="camera_joint" type="fixed">
+  <joint name="camera_joint_front" type="fixed">
     <parent link="base_link"/>
-    <child link="camera_link"/>
+    <child link="camera_link_front"/>
     <!-- front-top-ish: adjust as needed -->
     <origin xyz="0.25 0 0.15" rpy="0 0 0"/>
   </joint>
-  <link name="camera_link">
+  <link name="camera_link_front">
     <visual>
       <geometry>
@@ -28,14 +28,14 @@
   </link>
   <!-- Optical frame (REP-103/REP-105 style) -->
-  <joint name="camera_optical_joint" type="fixed">
-    <parent link="camera_link"/>
-    <child link="camera_link_optical"/>
+  <joint name="camera_optical_joint_front" type="fixed">
+    <parent link="camera_link_front"/>
+    <child link="camera_link_optical_front"/>
     <origin xyz="0 0 0" rpy="${-pi/2} 0 ${-pi/2}"/>
   </joint>
-  <link name="camera_link_optical"/>
+  <link name="camera_link_optical_front"/>
   <!-- Gazebo depth sensor -->
-  <gazebo reference="camera_link">
+  <gazebo reference="camera_link_front">
     <material>Gazebo/Red</material>
-    <sensor name="depth_camera" type="depth">
+    <sensor name="depth_camera_front" type="depth">
       <always_on>true</always_on>
       <visualize>true</visualize>
@@ -53,14 +53,14 @@
         </clip>
       </camera>
-      <plugin name="depth_camera_controller" filename="libgazebo_ros_camera.so">
+      <plugin name="depth_camera_front_controller" filename="libgazebo_ros_camera.so">
         <!-- frame published in CameraInfo -->
-        <frame_name>camera_link_optical</frame_name>
+        <frame_name>camera_link_optical_front</frame_name>
         <!-- predictable topic names -->
-        <camera_name>depth_camera</camera_name>
+        <camera_name>depth_camera_front</camera_name>
         <image_topic_name>rgb/image_raw</image_topic_name>
         <camera_info_topic_name>rgb/camera_info</camera_info_topic_name>
-        <depth_image_topic_name>depth/image_raw</depth_image_topic_name>
-        <depth_camera_info_topic_name>depth/camera_info</depth_camera_info_topic_name>
-        <point_cloud_topic_name>depth/points</point_cloud_topic_name>
+        <depth_image_topic_name>depth_camera_front/image_raw</depth_image_topic_name>
+        <depth_camera_info_topic_name>depth_camera_front/camera_info</depth_camera_info_topic_name>
+        <point_cloud_topic_name>depth_camera_front/points</point_cloud_topic_name>
       </plugin>
     </sensor>

File: qpl_ws/src/qpl_rover/description/rover.urdf.xacro (robot description, xacro)
@@ -8,5 +8,5 @@
     </xacro:if>
     <xacro:include filename="imu.xacro" />
-    <xacro:include filename="depth_camera.xacro" />
-    <xacro:include filename="back_camera.xacro" />
+    <xacro:include filename="depth_camera_front.xacro" />
+    <xacro:include filename="depth_camera_rear.xacro" />
 </robot>

Commit message: camera angle adjusted, need to filter out the ground

File: qpl_ws/src/qpl_rover/description/depth_camera_front.xacro (robot description, xacro)
@@ -6,5 +6,5 @@
     <child link="camera_link_front"/>
     <!-- front-top-ish: adjust as needed -->
-    <origin xyz="0.25 0 0.15" rpy="0 0 0"/>
+    <origin xyz="0.25 0 0.30" rpy="0 -0.18 0"/>
   </joint>
   <link name="camera_link_front">
@@ -50,5 +50,5 @@
         <clip>
           <near>0.05</near>
-          <far>8.0</far>
+          <far>5.0</far>
         </clip>
       </camera>

Commit message: front cam working for vslam

File: qpl_ws/src/qpl_rover/description/depth_camera_front.xacro (robot description, xacro)
@@ -6,5 +6,5 @@
     <child link="camera_link_front"/>
     <!-- front-top-ish: adjust as needed -->
-    <origin xyz="0.25 0 0.30" rpy="0 -0.18 0"/>
+    <origin xyz="0.25 0 0.15" rpy="0 0 0"/>
   </joint>
   <link name="camera_link_front">
@@ -50,5 +50,5 @@
         <clip>
           <near>0.05</near>
-          <far>5.0</far>
+          <far>8.0</far>
         </clip>
       </camera>

Commit message: urdf floating fixed

File: qpl_ws/src/qpl_rover/description/depth_camera_front.xacro (robot description, xacro)
@@ -6,5 +6,5 @@
     <child link="camera_link_front"/>
     <!-- front-top-ish: adjust as needed -->
-    <origin xyz="0.25 0 0.15" rpy="0 0 0"/>
+    <origin xyz="0.25 0 0.04" rpy="0 0 0"/>
   </joint>
   <link name="camera_link_front">

File: qpl_ws/src/qpl_rover/description/depth_camera_rear.xacro (robot description, xacro)
@@ -6,5 +6,5 @@
     <child link="camera_link_rear"/>
     <!-- front-top-ish: adjust as needed -->
-    <origin xyz="-0.25 0 0.15" rpy="0 0 ${pi}"/>
+    <origin xyz="-0.25 0 0.04" rpy="0 0 ${pi}"/>
   </joint>
   <link name="camera_link_rear">

File: qpl_ws/src/qpl_rover/description/imu.xacro (robot description, xacro)
@@ -14,5 +14,5 @@
       <parent link="${parent_link}"/>
       <child link="imu_link"/>
-      <origin xyz="0 0 0.15" rpy="0 0 0"/>
+      <origin xyz="0 0 0.0" rpy="0 0 0"/>
     </joint>
     <gazebo reference="imu_link">

File: qpl_ws/src/qpl_rover/description/rover_core.xacro (robot description, xacro)
@@ -2,57 +2,70 @@
 <robot xmlns:xacro="http://www.ros.org/wiki/xacro">
   <xacro:include filename="inertial_macros.xacro"/>
+  <!-- Materials -->
   <material name="gray"><color rgba="0.6 0.6 0.6 1.0"/></material>
   <material name="black"><color rgba="0.05 0.05 0.05 1.0"/></material>
   <material name="red"><color rgba="0.8 0.1 0.1 1.0"/></material>
   <material name="blue"><color rgba="0.2 0.2 1.0 1.0"/></material>
+  <!-- Base dimensions -->
   <xacro:property name="base_x" value="0.50"/>
   <xacro:property name="base_y" value="0.30"/>
   <xacro:property name="base_z" value="0.18"/>
+  <!-- Wheel dimensions -->
   <xacro:property name="wheel_r" value="0.10"/>
-  <!-- base_link is located above the ground by wheel radius + half the base height -->
-  <xacro:property name="base_z_origin" value="${wheel_r + base_z/2}"/>
   <xacro:property name="wheel_w" value="0.03"/>
+  <!-- Frame heights -->
+  <!-- base_footprint is on the ground -->
+  <!-- base_link is at chassis centre -->
+  <xacro:property name="base_link_z" value="${wheel_r + base_z/2}"/>
+  <!-- Wheel positions relative to base_link -->
   <xacro:property name="wheel_x_front" value="0.18"/>
   <xacro:property name="wheel_x_rear"  value="-0.18"/>
   <xacro:property name="wheel_y" value="${base_y/2 + wheel_w/2}"/>
-  <xacro:property name="wheel_z" value="${wheel_r}"/>
-  <!-- 2D ground-projected base frame -->
+  <xacro:property name="wheel_z" value="${-base_z/2}"/>
+  <!-- Ground-projected frame -->
   <link name="base_footprint"/>
-  <!-- Body frame -->
+  <!-- Main body frame -->
   <link name="base_link">
     <visual>
-      <origin xyz="0 0 ${base_z_origin}" rpy="0 0 0"/>
-      <geometry><box size="${base_x} ${base_y} ${base_z}"/></geometry>
+      <origin xyz="0 0 0" rpy="0 0 0"/>
+      <geometry>
+        <box size="${base_x} ${base_y} ${base_z}"/>
+      </geometry>
       <material name="gray"/>
     </visual>
     <collision>
-      <origin xyz="0 0 ${base_z_origin}" rpy="0 0 0"/>
-      <geometry><box size="${base_x} ${base_y} ${base_z}"/></geometry>
+      <origin xyz="0 0 0" rpy="0 0 0"/>
+      <geometry>
+        <box size="${base_x} ${base_y} ${base_z}"/>
+      </geometry>
     </collision>
     <xacro:inertial_box mass="10.0" x="${base_x}" y="${base_y}" z="${base_z}">
-      <origin xyz="0 0 ${base_z_origin}" rpy="0 0 0"/>
+      <origin xyz="0 0 0" rpy="0 0 0"/>
     </xacro:inertial_box>
   </link>
-  <!-- base_footprint -> base_link (base_link sits above ground) -->
+  <!-- Lift base_link above the ground -->
   <joint name="base_footprint_joint" type="fixed">
     <parent link="base_footprint"/>
     <child link="base_link"/>
-    <origin xyz="0 0 ${base_z_origin}" rpy="0 0 0"/>
+    <origin xyz="0 0 ${base_link_z}" rpy="0 0 0"/>
   </joint>
   <gazebo reference="base_link">
     <material>Gazebo/Grey</material>
   </gazebo>
-  <!-- WHEELS -->
+  <!-- Wheel macro -->
   <xacro:macro name="wheel_link" params="name">
     <link name="${name}">
       <visual>
         <origin xyz="0 0 0" rpy="${pi/2} 0 0"/>
-        <geometry><cylinder radius="${wheel_r}" length="${wheel_w}"/></geometry>
+        <geometry>
+          <cylinder radius="${wheel_r}" length="${wheel_w}"/>
+        </geometry>
         <material name="red"/>
       </visual>
-      <!-- slightly smaller collision helps avoid micro-binding -->
       <collision>
         <origin xyz="0 0 0" rpy="${pi/2} 0 0"/>
-        <geometry><cylinder radius="${wheel_r*0.98}" length="${wheel_w*0.95}"/></geometry>
+        <geometry>
+          <cylinder radius="${wheel_r*0.98}" length="${wheel_w*0.95}"/>
+        </geometry>
       </collision>
       <xacro:inertial_cylinder mass="0.5" length="${wheel_w}" radius="${wheel_r}">
@@ -63,19 +76,18 @@
       <material>Gazebo/Red</material>
     </gazebo>
-    <!-- ONE gazebo block per wheel -->
     <gazebo reference="${name}">
       <fdir1>1 0 0</fdir1>
-      <!-- skid-steer turning: reduce lateral friction -->
       <mu1>1.4</mu1>
       <mu2>0.2</mu2>
-      <!-- optional: allow lateral slip -->
       <slip1>0.0</slip1>
       <slip2>0.0</slip2>
     </gazebo>
   </xacro:macro>
+  <!-- Wheels -->
   <xacro:wheel_link name="front_left_wheel"/>
   <xacro:wheel_link name="front_right_wheel"/>
   <xacro:wheel_link name="rear_left_wheel"/>
   <xacro:wheel_link name="rear_right_wheel"/>
+  <!-- Wheel joints -->
   <joint name="front_left_wheel_joint" type="continuous">
     <parent link="base_link"/>

Commit message: updated rover model

File: qpl_ws/src/qpl_rover/description/depth_camera_front.xacro (robot description, xacro)
@@ -6,5 +6,5 @@
     <child link="camera_link_front"/>
     <!-- front-top-ish: adjust as needed -->
-    <origin xyz="0.25 0 0.04" rpy="0 0 0"/>
+    <origin xyz="0.2375 0 0.3525" rpy="0 0 0"/>
   </joint>
   <link name="camera_link_front">

File: qpl_ws/src/qpl_rover/description/depth_camera_rear.xacro (robot description, xacro)
@@ -6,5 +6,5 @@
     <child link="camera_link_rear"/>
     <!-- front-top-ish: adjust as needed -->
-    <origin xyz="-0.25 0 0.04" rpy="0 0 ${pi}"/>
+    <origin xyz="-0.2375 0 0.3525" rpy="0 0 ${pi}"/>
   </joint>
   <link name="camera_link_rear">

File: qpl_ws/src/qpl_rover/description/rover_core.xacro (robot description, xacro)
@@ -8,38 +8,50 @@
   <material name="blue"><color rgba="0.2 0.2 1.0 1.0"/></material>
   <!-- ========================================================= -->
-  <!-- Robot Dimensions                                          -->
-  <!-- Change these values and the rest of the robot updates      -->
-  <!-- ========================================================= -->
-  <!-- Base dimensions -->
-  <xacro:property name="base_x" value="0.50"/>
-  <xacro:property name="base_y" value="0.30"/>
-  <xacro:property name="base_z" value="0.18"/>
+  <!-- Main dimensions                                           -->
+  <!-- ========================================================= -->
+  <!-- Bottom cuboid -->
+  <xacro:property name="base_x" value="0.875"/>
+  <xacro:property name="base_y" value="0.599"/>
+  <xacro:property name="base_z" value="0.135"/>
+  <!-- Top trapezoid section -->
+  <!-- top_x smaller than base_x gives the trapezoid side profile -->
+  <xacro:property name="top_x" value="0.475"/>
+  <xacro:property name="top_y" value="${base_y}"/>
+  <xacro:property name="top_z" value="0.05"/>
+  <xacro:property name="trap_height" value="0.225"/>
+  <!-- Frame/support thickness -->
+  <xacro:property name="frame_t" value="0.04"/>
   <!-- Wheel dimensions -->
   <xacro:property name="wheel_r" value="0.15"/>
-  <xacro:property name="wheel_w" value="0.03"/>
-  <!-- Wheel placement scaling -->
-  <!-- How far from centre the wheels are along the robot length -->
-  <xacro:property name="wheel_x_offset" value="${base_x * 0.36}"/>
-  <!-- Small side clearance between chassis and wheel -->
+  <xacro:property name="wheel_w" value="0.15"/>
+  <!-- Wheel placement -->
+  <xacro:property name="wheel_x_offset" value="${base_x / 2}"/>
   <xacro:property name="wheel_side_clearance" value="0.00"/>
   <!-- ========================================================= -->
-  <!-- Derived dimensions                                        -->
-  <!-- Do not usually need to edit these                         -->
-  <!-- ========================================================= -->
-  <!-- base_footprint is on the ground -->
-  <!-- base_link is at chassis centre -->
+  <!-- Derived values                                            -->
+  <!-- ========================================================= -->
+  <!-- Base lift -->
   <xacro:property name="base_link_z" value="${wheel_r + base_z / 2}"/>
-  <!-- Wheel positions relative to base_link -->
+  <!-- Wheel positions -->
   <xacro:property name="wheel_x_front" value="${wheel_x_offset}"/>
   <xacro:property name="wheel_x_rear" value="${-wheel_x_offset}"/>
-  <!-- Wheels sit outside the chassis in Y -->
   <xacro:property name="wheel_y" value="${base_y / 2 + wheel_w / 2 + wheel_side_clearance}"/>
-  <!-- Wheel centre is level with bottom of chassis -->
-  <!-- This means wheel bottom touches ground because base_link is lifted by wheel_r + base_z/2 -->
   <xacro:property name="wheel_z" value="${-base_z / 2}"/>
+  <!-- Top deck position -->
+  <xacro:property name="top_deck_z" value="${base_z / 2 + trap_height + top_z / 2}"/>
+  <!-- Slanted support geometry -->
+  <xacro:property name="support_dx" value="${(base_x - top_x) / 2}"/>
+  <xacro:property name="support_len" value="${math.sqrt(support_dx * support_dx + trap_height * trap_height)}"/>
+  <xacro:property name="support_pitch" value="${math.atan2(trap_height, support_dx)}"/>
+  <!-- Centres of support beams -->
+  <xacro:property name="support_front_x" value="${(base_x + top_x) / 4}"/>
+  <xacro:property name="support_rear_x" value="${-support_front_x}"/>
+  <xacro:property name="support_y" value="${base_y / 2 - frame_t / 2}"/>
+  <xacro:property name="support_z" value="${base_z / 2 + trap_height / 2}"/>
   <!-- ========================================================= -->
   <!-- Base frames                                               -->
   <!-- ========================================================= -->
   <link name="base_footprint"/>
+  <!-- Bottom cuboid -->
   <link name="base_link">
     <visual>
@@ -60,5 +72,4 @@
     </xacro:inertial_box>
   </link>
-  <!-- Lift base_link above the ground -->
   <joint name="base_footprint_joint" type="fixed">
     <parent link="base_footprint"/>
@@ -70,4 +81,66 @@
   </gazebo>
   <!-- ========================================================= -->
+  <!-- Generic box member macro                                  -->
+  <!-- ========================================================= -->
+  <xacro:macro name="box_member" params="name sx sy sz mass colour">
+    <link name="${name}">
+      <visual>
+        <origin xyz="0 0 0" rpy="0 0 0"/>
+        <geometry>
+          <box size="${sx} ${sy} ${sz}"/>
+        </geometry>
+        <material name="${colour}"/>
+      </visual>
+      <collision>
+        <origin xyz="0 0 0" rpy="0 0 0"/>
+        <geometry>
+          <box size="${sx} ${sy} ${sz}"/>
+        </geometry>
+      </collision>
+      <xacro:inertial_box mass="${mass}" x="${sx}" y="${sy}" z="${sz}">
+        <origin xyz="0 0 0" rpy="0 0 0"/>
+      </xacro:inertial_box>
+    </link>
+    <gazebo reference="${name}">
+      <material>Gazebo/Grey</material>
+    </gazebo>
+  </xacro:macro>
+  <!-- ========================================================= -->
+  <!-- Upper trapezoid section                                   -->
+  <!-- ========================================================= -->
+  <!-- Top deck -->
+  <xacro:box_member name="top_deck" sx="${top_x}" sy="${top_y}" sz="${top_z}" mass="2.0" colour="blue"/>
+  <joint name="top_deck_joint" type="fixed">
+    <parent link="base_link"/>
+    <child link="top_deck"/>
+    <origin xyz="0 0 ${top_deck_z}" rpy="0 0 0"/>
+  </joint>
+  <!-- Front supports -->
+  <xacro:box_member name="front_left_support"  sx="${support_len}" sy="${frame_t}" sz="${frame_t}" mass="0.5" colour="black"/>
+  <xacro:box_member name="front_right_support" sx="${support_len}" sy="${frame_t}" sz="${frame_t}" mass="0.5" colour="black"/>
+  <joint name="front_left_support_joint" type="fixed">
+    <parent link="base_link"/>
+    <child link="front_left_support"/>
+    <origin xyz="${support_front_x} ${support_y} ${support_z}" rpy="0 ${support_pitch} 0"/>
+  </joint>
+  <joint name="front_right_support_joint" type="fixed">
+    <parent link="base_link"/>
+    <child link="front_right_support"/>
+    <origin xyz="${support_front_x} -${support_y} ${support_z}" rpy="0 ${support_pitch} 0"/>
+  </joint>
+  <!-- Rear supports -->
+  <xacro:box_member name="rear_left_support"  sx="${support_len}" sy="${frame_t}" sz="${frame_t}" mass="0.5" colour="black"/>
+  <xacro:box_member name="rear_right_support" sx="${support_len}" sy="${frame_t}" sz="${frame_t}" mass="0.5" colour="black"/>
+  <joint name="rear_left_support_joint" type="fixed">
+    <parent link="base_link"/>
+    <child link="rear_left_support"/>
+    <origin xyz="${support_rear_x} ${support_y} ${support_z}" rpy="0 -${support_pitch} 0"/>
+  </joint>
+  <joint name="rear_right_support_joint" type="fixed">
+    <parent link="base_link"/>
+    <child link="rear_right_support"/>
+    <origin xyz="${support_rear_x} -${support_y} ${support_z}" rpy="0 -${support_pitch} 0"/>
+  </joint>
+  <!-- ========================================================= -->
   <!-- Wheel macro                                               -->
   <!-- ========================================================= -->
@@ -75,5 +148,4 @@
     <link name="${name}">
       <visual>
-        <!-- Cylinder is rotated so its axle runs along Y -->
         <origin xyz="0 0 0" rpy="${pi / 2} 0 0"/>
         <geometry>

Commit message: adjusted xacro files to real measurements for chassis and cameras

File: qpl_ws/src/qpl_rover/description/depth_camera_front.xacro (robot description, xacro)
@@ -6,5 +6,5 @@
     <child link="camera_link_front"/>
     <!-- front-top-ish: adjust as needed -->
-    <origin xyz="0.2375 0 0.3525" rpy="0 0 0"/>
+    <origin xyz="0.265 0 0.26" rpy="0 0 0"/>
   </joint>
   <link name="camera_link_front">

File: qpl_ws/src/qpl_rover/description/depth_camera_rear.xacro (robot description, xacro)
@@ -6,5 +6,5 @@
     <child link="camera_link_rear"/>
     <!-- front-top-ish: adjust as needed -->
-    <origin xyz="-0.2375 0 0.3525" rpy="0 0 ${pi}"/>
+    <origin xyz="-0.265 0 0.3" rpy="0 0 ${pi}"/>
   </joint>
   <link name="camera_link_rear">

File: qpl_ws/src/qpl_rover/description/rover_core.xacro (robot description, xacro)
@@ -11,12 +11,12 @@
   <!-- ========================================================= -->
   <!-- Bottom cuboid -->
-  <xacro:property name="base_x" value="0.875"/>
-  <xacro:property name="base_y" value="0.5806"/>
-  <xacro:property name="base_z" value="0.135"/>
+  <xacro:property name="base_x" value="0.925"/>
+  <xacro:property name="base_y" value="0.745"/>
+  <xacro:property name="base_z" value="0.025"/>
   <!-- Top trapezoid section -->
   <!-- top_x smaller than base_x gives the trapezoid side profile -->
-  <xacro:property name="top_x" value="0.475"/>
+  <xacro:property name="top_x" value="0.53"/>
   <xacro:property name="top_y" value="${base_y}"/>
-  <xacro:property name="top_z" value="0.05"/>
+  <xacro:property name="top_z" value="${base_z}"/>
   <xacro:property name="trap_height" value="0.225"/>
   <!-- Frame/support thickness -->

Commit message: Set physical simulation parameters to near-final values

File: qpl_ws/src/qpl_rover/description/depth_camera_front.xacro (robot description, xacro)
@@ -5,6 +5,5 @@
     <parent link="base_link"/>
     <child link="camera_link_front"/>
-    <!-- front-top-ish: adjust as needed -->
-    <origin xyz="0.265 0 0.26" rpy="0 0 0"/>
+    <origin xyz="0.465 0 0.02" rpy="0 0 0"/>
   </joint>
   <link name="camera_link_front">

File: qpl_ws/src/qpl_rover/description/depth_camera_rear.xacro (robot description, xacro)
@@ -5,6 +5,5 @@
     <parent link="base_link"/>
     <child link="camera_link_rear"/>
-    <!-- front-top-ish: adjust as needed -->
-    <origin xyz="-0.265 0 0.3" rpy="0 0 ${pi}"/>
+    <origin xyz="-0.465 0 0.02" rpy="0 0 0"/>
   </joint>
   <link name="camera_link_rear">
