Commit message: Sim: Gazebo Harmonic with terramechanics sand on the US arena
Moves the sim from Gazebo Classic to Gazebo Harmonic so the wheels can run on
simulated sand: the gz_terramechanics plugin (Bekker-Wong wheel-soil model)
replaces rigid-ground friction on the arena floor with sinkage and
slip-dependent traction, using lunar soil parameters.

- Vendor gz_terramechanics (GPL-3.0), patched for our wheels (axis direction
  from config instead of wheel names), NaN-free when a wheel stops, and an
  ament build with OpenMP and a plugin-path hook.
- URDF: gz_ros2_control, Harmonic IMU and cameras (depth sensors become
  rgbd_camera so VO still gets registered colour), wheel contact sensors and
  the plugin, sim_mode only. Real-rover URDF unchanged.
- us_arena_terrain.world ported (same layout, PBR AprilTag); sim.launch.py
  uses ros_gz with the same ROS topic names, and bridges the world clock.
- Install script, GZ_VERSION export and sim.repos for gz_ros2_control.
- test/sim/sand_sim_check.py smoke test.

File: qpl_ws/src/qpl_rover/description/depth_camera_front.xacro (robot description, xacro)
@@ -51,8 +51,11 @@
       <visualize>true</visualize>
       <update_rate>10</update_rate>
+      <!-- camera_info goes to the sibling .../camera_info topic -->
+      <topic>depth_camera_front/image_raw</topic>
+      <gz_frame_id>camera_link_optical_front</gz_frame_id>
       <camera>
         <horizontal_fov>1.51844</horizontal_fov>
         <image>
-          <format>B8G8R8</format>
+          <format>R8G8B8</format>
           <width>1280</width>
           <height>720</height>
@@ -63,19 +66,21 @@
         </clip>
       </camera>
-      <plugin name="camera_front_color_controller" filename="libgazebo_ros_camera.so">
-        <frame_name>camera_link_optical_front</frame_name>
-        <camera_name>depth_camera_front</camera_name>
-      </plugin>
     </sensor>
     <!-- Depth camera: 480p point cloud for the Nav2 voxel layer (mirrors the front
          RealSense depth at 848x480). -->
-    <sensor name="depth_camera_front" type="depth">
+    <!-- rgbd_camera, not depth_camera: Harmonic's depth_camera only outputs depth, and the
+         visual odometry needs a colour image registered with it (same resolution,
+         intrinsics and frame), which gazebo_ros's depth camera used to publish. -->
+    <sensor name="depth_camera_front" type="rgbd_camera">
       <always_on>true</always_on>
       <visualize>true</visualize>
       <update_rate>10</update_rate>
+      <!-- publishes depth_camera_front_depth/image (colour), /depth_image, /camera_info, /points -->
+      <topic>depth_camera_front_depth</topic>
+      <gz_frame_id>camera_link_optical_front</gz_frame_id>
       <camera>
         <horizontal_fov>1.51844</horizontal_fov>
         <image>
-          <format>B8G8R8</format>
+          <format>R8G8B8</format>
           <width>848</width>
           <height>480</height>
@@ -86,8 +91,4 @@
         </clip>
       </camera>
-      <plugin name="depth_camera_front_controller" filename="libgazebo_ros_camera.so">
-        <frame_name>camera_link_optical_front</frame_name>
-        <camera_name>depth_camera_front_depth</camera_name>
-      </plugin>
     </sensor>
   </gazebo>

File: qpl_ws/src/qpl_rover/description/depth_camera_rear.xacro (robot description, xacro)
@@ -50,9 +50,12 @@
       <visualize>true</visualize>
       <update_rate>10</update_rate>
+      <!-- camera_info goes to the sibling .../camera_info topic -->
+      <topic>depth_camera_rear/image_raw</topic>
+      <gz_frame_id>camera_link_optical_rear</gz_frame_id>
       <camera>
         <horizontal_fov>1.019272</horizontal_fov>
         <vertical_fov>2</vertical_fov>
         <image>
-          <format>B8G8R8</format>
+          <format>R8G8B8</format>
           <width>1280</width>
           <height>720</height>
@@ -63,20 +66,22 @@
         </clip>
       </camera>
-      <plugin name="camera_rear_color_controller" filename="libgazebo_ros_camera.so">
-        <frame_name>camera_link_optical_rear</frame_name>
-        <camera_name>depth_camera_rear</camera_name>
-      </plugin>
     </sensor>
     <!-- Depth camera: 480p point cloud for the Nav2 voxel layer (mirrors the rear
          Orbbec depth at 640x480). -->
-    <sensor name="depth_camera_rear" type="depth">
+    <!-- rgbd_camera, not depth_camera: Harmonic's depth_camera only outputs depth, and the
+         visual odometry needs a colour image registered with it (same resolution,
+         intrinsics and frame), which gazebo_ros's depth camera used to publish. -->
+    <sensor name="depth_camera_rear" type="rgbd_camera">
       <always_on>true</always_on>
       <visualize>true</visualize>
       <update_rate>10</update_rate>
+      <!-- publishes depth_camera_rear_depth/image (colour), /depth_image, /camera_info, /points -->
+      <topic>depth_camera_rear_depth</topic>
+      <gz_frame_id>camera_link_optical_rear</gz_frame_id>
       <camera>
         <horizontal_fov>1.019272</horizontal_fov>
         <vertical_fov>2</vertical_fov>
         <image>
-          <format>B8G8R8</format>
+          <format>R8G8B8</format>
           <width>640</width>
           <height>480</height>
@@ -87,8 +92,4 @@
         </clip>
       </camera>
-      <plugin name="depth_camera_rear_controller" filename="libgazebo_ros_camera.so">
-        <frame_name>camera_link_optical_rear</frame_name>
-        <camera_name>depth_camera_rear_depth</camera_name>
-      </plugin>
     </sensor>
   </gazebo>

File: qpl_ws/src/qpl_rover/description/imu.xacro (robot description, xacro)
@@ -21,6 +21,12 @@
         <update_rate>50</update_rate>
         <visualize>false</visualize>
-        <topic>imu</topic>
+        <topic>imu/data</topic>
+        <!-- imu_link is folded into base_link when the URDF becomes SDF, so name the frame -->
+        <gz_frame_id>imu_link</gz_frame_id>
         <imu>
+          <!-- orientation relative to the world, like the old initial_orientation_as_reference false -->
+          <orientation_reference_frame>
+            <localization>ENU</localization>
+          </orientation_reference_frame>
           <angular_velocity>
             <x>
@@ -76,11 +82,4 @@
           </linear_acceleration>
         </imu>
-        <plugin name="imu_plugin" filename="libgazebo_ros_imu_sensor.so">
-          <ros>
-            <remapping>~/out:=/imu/data</remapping>
-          </ros>
-          <frame_name>imu_link</frame_name>
-          <initial_orientation_as_reference>false</initial_orientation_as_reference>
-        </plugin>
       </sensor>
     </gazebo>

File: qpl_ws/src/qpl_rover/description/ros2_control.xacro (robot description, xacro)
@@ -59,5 +59,5 @@
         <ros2_control name="GazeboSystem" type="system">
             <hardware>
-                <plugin>gazebo_ros2_control/GazeboSystem</plugin>
+                <plugin>gz_ros2_control/GazeboSimSystem</plugin>
             </hardware>
             <joint name="front_left_wheel_joint">
@@ -118,5 +118,5 @@
     </xacro:if>
     <gazebo>
-        <plugin name="gazebo_ros2_control" filename="libgazebo_ros2_control.so">
+        <plugin name="gz_ros2_control::GazeboSimROS2ControlPlugin" filename="gz_ros2_control-system">
             <parameters>$(find qpl_rover)/config/my_controllers.yaml</parameters>
             <parameters>$(find qpl_rover)/config/gaz_ros2_ctl_use_sim.yaml</parameters>

File: qpl_ws/src/qpl_rover/description/rover_core.xacro (robot description, xacro)
@@ -411,4 +411,6 @@
       <material>Gazebo/Red</material>
     </gazebo>
+    <!-- Friction against anything that isn't sand (boulders, walls). On the sand the
+         terramechanics plugin zeroes it and applies its own traction instead. -->
     <gazebo reference="${name}">
       <fdir1>1 0 0</fdir1>
@@ -418,4 +420,28 @@
       <slip2>0.0</slip2>
     </gazebo>
+    <!-- The terramechanics plugin reads each wheel's load from this sensor. The URDF to
+         SDF conversion names a link's collisions <link>_collision, <link>_collision_1, ...;
+         sim_mode has the centre cylinder plus 10 tyre edge slices. -->
+    <xacro:if value="$(arg sim_mode)">
+      <gazebo reference="${name}">
+        <sensor name="${name}_contact" type="contact">
+          <always_on>true</always_on>
+          <update_rate>1000</update_rate>
+          <contact>
+            <collision>${name}_collision</collision>
+            <collision>${name}_collision_1</collision>
+            <collision>${name}_collision_2</collision>
+            <collision>${name}_collision_3</collision>
+            <collision>${name}_collision_4</collision>
+            <collision>${name}_collision_5</collision>
+            <collision>${name}_collision_6</collision>
+            <collision>${name}_collision_7</collision>
+            <collision>${name}_collision_8</collision>
+            <collision>${name}_collision_9</collision>
+            <collision>${name}_collision_10</collision>
+          </contact>
+        </sensor>
+      </gazebo>
+    </xacro:if>
   </xacro:macro>
   <!-- ========================================================= -->
@@ -492,9 +518,10 @@
   <xacro:wheel_mount name="rear_right_wheel"
       xyz="${-top_long_len / 2 - bar_t / 2} ${-wheel_support_len / 2} ${-lower_support_len - bar_t}"/>
-  <!-- The sand joints aren't ros2_control joints, so publish their state for TF. -->
+  <!-- The sand joints aren't ros2_control joints, so publish their state for TF
+       (sim.launch.py bridges sand_joint_states onto /joint_states). -->
   <xacro:if value="$(arg sim_mode)">
     <gazebo>
-      <plugin name="sand_joint_states" filename="libgazebo_ros_joint_state_publisher.so">
-        <update_rate>50</update_rate>
+      <plugin name="gz::sim::systems::JointStatePublisher" filename="gz-sim-joint-state-publisher-system">
+        <topic>sand_joint_states</topic>
         <joint_name>front_left_wheel_sand_joint</joint_name>
         <joint_name>front_right_wheel_sand_joint</joint_name>
@@ -503,4 +530,11 @@
       </plugin>
     </gazebo>
+    <!-- Wheel-soil forces (sinkage, slip-dependent traction, lateral shear) from Bekker-Wong
+         terramechanics. Wheel geometry and the soil are in config/terramechanics. -->
+    <gazebo>
+      <plugin name="gz_terramechanics::TerramechanicsSystem" filename="TerramechanicsSystem">
+        <config_path>$(find qpl_rover)/config/terramechanics</config_path>
+      </plugin>
+    </gazebo>
   </xacro:if>
 </robot>
