Commit message: updated nav2

File: qpl_ws/src/qpl_rover/description/depth_camera_rear.xacro (robot description, xacro)
@@ -6,5 +6,5 @@
     <child link="camera_link_rear"/>
     <!-- front-top-ish: adjust as needed -->
-    <origin xyz="-0.25 0 0.15" rpy="0 0 0"/>
+    <origin xyz="-0.25 0 0.15" rpy="0 0 ${pi}"/>
   </joint>
   <link name="camera_link_rear">

Commit message: Clean-up of physical parameters and nav changed back to native voxellayer.

File: qpl_ws/src/qpl_rover/description/depth_camera_rear.xacro (robot description, xacro)
@@ -5,5 +5,5 @@
     <parent link="base_link"/>
     <child link="camera_link_rear"/>
-    <origin xyz="-0.465 0 0.02" rpy="0 0 0"/>
+    <origin xyz="-0.465 0 0.02" rpy="0 0 ${pi}"/>
   </joint>
   <link name="camera_link_rear">
