Commit message: arduino serial added

File: qpl_ws/src/qpl_rover/description/ros2_control.xacro (robot description, xacro)
@@ -1,4 +1,34 @@
 <?xml version="1.0"?>
 <robot xmlns:xacro="http://www.ros.org/wiki/xacro">
+  <xacro:unless value="$(arg sim_mode)">
+      <ros2_control name="RealRobot" type="system">
+          <hardware>
+              <plugin>diffdrive_arduino/DiffDriveArduino</plugin>
+              <param name="left_wheel_name">left_wheel_joint</param>
+              <param name="right_wheel_name">right_wheel_joint</param>
+              <param name="loop_rate">30</param>
+              <param name="device">/dev/ttyUSB0</param>
+              <param name="baud_rate">57600</param>
+              <param name="timeout">1000</param>
+              <param name="enc_counts_per_rev">3436</param>
+          </hardware>
+          <joint name="left_wheel_joint">
+              <command_interface name="velocity">
+                  <param name="min">-10</param>
+                  <param name="max">10</param>
+              </command_interface>
+              <state_interface name="velocity"/>
+              <state_interface name="position"/>
+          </joint>
+          <joint name="right_wheel_joint">
+              <command_interface name="velocity">
+                  <param name="min">-10</param>
+                  <param name="max">10</param>
+              </command_interface>
+              <state_interface name="velocity"/>
+              <state_interface name="position"/>
+          </joint>
+      </ros2_control>
+  </xacro:unless>
   <xacro:if value="$(arg sim_mode)">
     <ros2_control name="GazeboSystem" type="system">

File: qpl_ws/src/qpl_rover/description/rover.urdf.xacro (robot description, xacro)
@@ -2,5 +2,5 @@
 <robot xmlns:xacro="http://www.ros.org/wiki/xacro"  name="robot">
     <xacro:arg name="use_ros2_control" default="true"/>
-    <xacro:arg name="sim_mode" default="true"/>
+    <xacro:arg name="sim_mode" default="false"/>
     <xacro:include filename="rover_core.xacro" />
     <xacro:if value="$(arg use_ros2_control)">

Commit message: hardware interface connection made

File: qpl_ws/src/qpl_rover/description/ros2_control.xacro (robot description, xacro)
@@ -2,7 +2,7 @@
 <robot xmlns:xacro="http://www.ros.org/wiki/xacro">
   <xacro:unless value="$(arg sim_mode)">
-      <ros2_control name="RealRobot" type="system">
+      <ros2_control name="RealRover" type="system">
           <hardware>
-              <plugin>diffdrive_arduino/DiffDriveArduino</plugin>
+              <plugin>diffdrive_arduino/DiffDriveArduinoHardware</plugin>
               <param name="left_wheel_name">left_wheel_joint</param>
               <param name="right_wheel_name">right_wheel_joint</param>
@@ -13,21 +13,37 @@
               <param name="enc_counts_per_rev">3436</param>
           </hardware>
-          <joint name="left_wheel_joint">
-              <command_interface name="velocity">
-                  <param name="min">-10</param>
-                  <param name="max">10</param>
-              </command_interface>
-              <state_interface name="velocity"/>
-              <state_interface name="position"/>
-          </joint>
-          <joint name="right_wheel_joint">
-              <command_interface name="velocity">
-                  <param name="min">-10</param>
-                  <param name="max">10</param>
-              </command_interface>
-              <state_interface name="velocity"/>
-              <state_interface name="position"/>
-          </joint>
-      </ros2_control>
+      <joint name="front_left_wheel_joint">
+        <command_interface name="velocity">
+            <param name="min_velocity">-10</param>
+            <param name="max_velocity">10</param>
+        </command_interface>
+        <state_interface name="position"/>
+        <state_interface name="velocity"/>
+      </joint>
+      <joint name="front_right_wheel_joint">
+        <command_interface name="velocity">
+            <param name="min_velocity">-10</param>
+            <param name="max_velocity">10</param>
+        </command_interface>
+        <state_interface name="position"/>
+        <state_interface name="velocity"/>
+      </joint>
+      <joint name="rear_left_wheel_joint">
+        <command_interface name="velocity">
+              <param name="min_velocity">-10</param>
+              <param name="max_velocity">10</param>
+        </command_interface>
+        <state_interface name="position"/>
+        <state_interface name="velocity"/>
+      </joint>
+      <joint name="rear_right_wheel_joint">
+        <command_interface name="velocity">
+              <param name="min_velocity">-10</param>
+              <param name="max_velocity">10</param>
+        </command_interface>
+        <state_interface name="position"/>
+        <state_interface name="velocity"/>
+      </joint>
+    </ros2_control>
   </xacro:unless>
   <xacro:if value="$(arg sim_mode)">

Commit message: motor feedback added

File: qpl_ws/src/qpl_rover/description/ros2_control.xacro (robot description, xacro)
@@ -19,4 +19,5 @@
               <param name="gear_ratio">100</param>
               <param name="loopback_mode">false</param>
+              <param name="feedback_enabled">true</param>
               <param name="print_commands">false</param>
               <param name="print_status">false</param>

File: qpl_ws/src/qpl_rover/description/rover_core.xacro (robot description, xacro)
@@ -12,5 +12,5 @@
   <xacro:property name="base_z" value="0.18"/>
   <!-- Wheel dimensions -->
-  <xacro:property name="wheel_r" value="0.10"/>
+  <xacro:property name="wheel_r" value="0.15"/>
   <xacro:property name="wheel_w" value="0.03"/>
   <!-- Frame heights -->

Commit message: drum sim

File: qpl_ws/src/qpl_rover/description/ros2_control.xacro (robot description, xacro)
@@ -91,4 +91,17 @@
         <state_interface name="velocity"/>
       </joint>
+      <joint name="drum_joint">
+        <command_interface name="velocity">
+          <param name="min_velocity">-0.1</param>
+          <param name="max_velocity">0.1</param>
+        </command_interface>
+          <state_interface name="position"/>
+          <state_interface name="velocity"/>
+      </joint>
+            <joint name="drum_spin_joint">
+        <command_interface name="velocity"/>
+          <state_interface name="position"/>
+          <state_interface name="velocity"/>
+      </joint>
     </ros2_control>
   </xacro:if>

File: qpl_ws/src/qpl_rover/description/rover_core.xacro (robot description, xacro)
@@ -114,3 +114,75 @@
     <axis xyz="0 1 0"/>
   </joint>
+<!-- Drum (placeholder primitive, prismatic lift + continuous spin) -->
+  <xacro:property name="drum_radius" value="0.10"/>
+  <xacro:property name="drum_length" value="0.30"/>
+  <xacro:property name="drum_mass"   value="1.0"/>
+  <!-- Mount at middle of chassis -->
+  <xacro:property name="drum_x" value="${base_x/2 + drum_radius + 0.1}"/>
+  <xacro:property name="drum_y" value="0.0"/>
+  <xacro:property name="drum_z" value="${base_z/2 + drum_radius - 0.1}"/>
+  <!-- Drum lift travel: 0 = up (rest), -0.1 = lowered -->
+  <xacro:property name="drum_lift_lower" value="-0.1"/>
+  <xacro:property name="drum_lift_upper" value="0.0"/>
+  <xacro:property name="drum_lift_effort" value="40.0"/>
+  <xacro:property name="drum_lift_velocity" value="0.1"/>
+  <!-- Drum spin limits -->
+  <xacro:property name="drum_spin_effort" value="50.0"/>
+  <xacro:property name="drum_spin_velocity" value="10.0"/>
+  <!-- Intermediate frame -->
+<link name="drum_lift_link">
+  <inertial>
+    <origin xyz="0 0 0" rpy="0 0 0"/>
+    <mass value="2.0"/>
+    <inertia ixx="0.01" ixy="0" ixz="0" iyy="0.01" iyz="0" izz="0.01"/>
+  </inertial>
+</link>
+  <!-- Actual drum link: visual, collision, real inertia -->
+  <link name="drum_link">
+    <visual>
+      <origin xyz="0 0 0" rpy="${pi/2} 0 0"/>
+      <geometry>
+        <cylinder radius="${drum_radius}" length="${drum_length}"/>
+      </geometry>
+      <material name="blue"/>
+    </visual>
+    <collision>
+      <origin xyz="0 0 0" rpy="${pi/2} 0 0"/>
+      <geometry>
+        <cylinder radius="${drum_radius}" length="${drum_length}"/>
+      </geometry>
+    </collision>
+    <xacro:inertial_cylinder mass="${drum_mass}" length="${drum_length}" radius="${drum_radius}">
+      <origin xyz="0 0 0" rpy="0 0 0"/>
+    </xacro:inertial_cylinder>
+  </link>
+  <!-- Lift joint: prismatic along Z. Origin stays at base_link,
+       offset moved down to drum_spin_joint.  change to type prismatic -->
+  <joint name="drum_joint" type="prismatic">
+    <parent link="base_link"/>
+    <child link="drum_lift_link"/>
+    <origin xyz="0 0 0" rpy="0 0 0"/>
+    <axis xyz="0 0 1"/>
+    <limit lower="${drum_lift_lower}"
+           upper="${drum_lift_upper}"
+           effort="${drum_lift_effort}"
+           velocity="${drum_lift_velocity}"/>
+    <dynamics damping="5.0" friction="50.0"/>
+  </joint>
+  <!-- Spin joint: continuous around Y. Carries the X/Z offset
+       that places the drum at the front of the rover. -->
+  <joint name="drum_spin_joint" type="continuous">
+    <parent link="drum_lift_link"/>
+    <child link="drum_link"/>
+    <origin xyz="${drum_x} ${drum_y} ${drum_z}" rpy="0 0 0"/>
+    <axis xyz="0 1 0"/>
+    <limit effort="${drum_spin_effort}" velocity="${drum_spin_velocity}"/>
+    <dynamics damping="0.1" friction="0.05"/>
+  </joint>
+  <gazebo reference="drum_link">
+    <material>Gazebo/Blue</material>
+  </gazebo>
+  <gazebo>
+  <self_collide>0</self_collide>
+  </gazebo>
 </robot>

Commit message: drum update

File: qpl_ws/src/qpl_rover/description/ros2_control.xacro (robot description, xacro)
@@ -96,7 +96,7 @@
       </joint>
       <joint name="drum_joint">
-        <command_interface name="velocity">
-          <param name="min_velocity">-0.1</param>
-          <param name="max_velocity">0.1</param>
+        <command_interface name="position">
+          <param name="min">0.0</param>
+          <param name="max">1.0</param>
         </command_interface>
           <state_interface name="position"/>

File: qpl_ws/src/qpl_rover/description/rover.urdf.xacro (robot description, xacro)
@@ -4,4 +4,5 @@
     <xacro:arg name="sim_mode" default="false"/>
     <xacro:include filename="rover_core.xacro" />
+    <xacro:include filename="drum_bucket.xacro" />
     <xacro:if value="$(arg use_ros2_control)">
         <xacro:include filename="ros2_control.xacro" />

File: qpl_ws/src/qpl_rover/description/rover_core.xacro (robot description, xacro)
@@ -209,75 +209,3 @@
     <axis xyz="0 1 0"/>
   </joint>
-<!-- Drum (placeholder primitive, prismatic lift + continuous spin) -->
-  <xacro:property name="drum_radius" value="0.10"/>
-  <xacro:property name="drum_length" value="0.30"/>
-  <xacro:property name="drum_mass"   value="1.0"/>
-  <!-- Mount at middle of chassis -->
-  <xacro:property name="drum_x" value="${base_x/2 - 0.5}"/>
-  <xacro:property name="drum_y" value="0.0"/>
-  <xacro:property name="drum_z" value="${base_z/2 + drum_radius + 0.8}"/>
-  <!-- Drum lift travel: 0 = up (rest), -0.1 = lowered -->
-  <xacro:property name="drum_lift_lower" value="-0.1"/>
-  <xacro:property name="drum_lift_upper" value="0.0"/>
-  <xacro:property name="drum_lift_effort" value="40.0"/>
-  <xacro:property name="drum_lift_velocity" value="0.1"/>
-  <!-- Drum spin limits -->
-  <xacro:property name="drum_spin_effort" value="50.0"/>
-  <xacro:property name="drum_spin_velocity" value="10.0"/>
-  <!-- Intermediate frame -->
-<link name="drum_lift_link">
-  <inertial>
-    <origin xyz="0 0 0" rpy="0 0 0"/>
-    <mass value="2.0"/>
-    <inertia ixx="0.01" ixy="0" ixz="0" iyy="0.01" iyz="0" izz="0.01"/>
-  </inertial>
-</link>
-  <!-- Actual drum link: visual, collision, real inertia -->
-  <link name="drum_link">
-    <visual>
-      <origin xyz="0 0 0" rpy="0 0 0"/>
-      <geometry>
-        <box size="${2*drum_radius} ${drum_length} ${2*drum_radius}"/>
-      </geometry>
-      <material name="blue"/>
-    </visual>
-    <collision>
-      <origin xyz="0 0 0" rpy="0 0 0"/>
-      <geometry>
-        <box size="${2*drum_radius} ${drum_length} ${2*drum_radius}"/>
-      </geometry>
-    </collision>
-    <xacro:inertial_cylinder mass="${drum_mass}" length="${drum_length}" radius="${drum_radius}">
-      <origin xyz="0 0 0" rpy="0 0 0"/>
-    </xacro:inertial_cylinder>
-  </link>
-  <!-- Lift joint: prismatic along Z. Origin stays at base_link,
-       offset moved down to drum_spin_joint.  change to type prismatic -->
-  <joint name="drum_joint" type="prismatic">
-    <parent link="base_link"/>
-    <child link="drum_lift_link"/>
-    <origin xyz="0 0 0" rpy="0 0 0"/>
-    <axis xyz="0 0 1"/>
-    <limit lower="${drum_lift_lower}"
-           upper="${drum_lift_upper}"
-           effort="${drum_lift_effort}"
-           velocity="${drum_lift_velocity}"/>
-    <dynamics damping="5.0" friction="50.0"/>
-  </joint>
-  <!-- Spin joint: continuous around Y. Carries the X/Z offset
-       that places the drum at the front of the rover. -->
-  <joint name="drum_spin_joint" type="continuous">
-    <parent link="drum_lift_link"/>
-    <child link="drum_link"/>
-    <origin xyz="${drum_x} ${drum_y} ${drum_z}" rpy="0 0 0"/>
-    <axis xyz="0 1 0"/>
-    <limit effort="${drum_spin_effort}" velocity="${drum_spin_velocity}"/>
-    <dynamics damping="0.1" friction="0.05"/>
-  </joint>
-  <gazebo reference="drum_link">
-    <material>Gazebo/Blue</material>
-  </gazebo>
-  <gazebo>
-  <self_collide>0</self_collide>
-  </gazebo>
 </robot>
