Commit message: Corrections to xacro

File: qpl_ws/src/qpl_rover/description/ros2_control.xacro (robot description, xacro)
@@ -38,8 +38,7 @@
                 <state_interface name="velocity"/>
             </joint>
-            <!-- 0.0 = retract, 0.5 = stop, 1.0 = extend -->
             <joint name="left_linear_actuator_joint">
                 <command_interface name="position">
-                    <param name="min">0.0</param>
+                    <param name="min">-1.0</param>
                     <param name="max">1.0</param>
                 </command_interface>
@@ -48,5 +47,5 @@
             <joint name="right_linear_actuator_joint">
                 <command_interface name="position">
-                    <param name="min">0.0</param>
+                    <param name="min">-1.0</param>
                     <param name="max">1.0</param>
                 </command_interface>
@@ -54,5 +53,8 @@
             </joint>
             <joint name="drum_spin_joint">
-                <command_interface name="velocity"/>
+                <command_interface name="velocity">
+                    <param name="min_velocity">-10</param>
+                    <param name="max_velocity">10</param>
+                </command_interface>
                 <state_interface name="position"/>
                 <state_interface name="velocity"/>
@@ -97,13 +99,7 @@
                 <state_interface name="velocity"/>
             </joint>
-            <joint name="drum_spin_joint">
-                <command_interface name="velocity"/>
-                <state_interface name="position"/>
-                <state_interface name="velocity"/>
-            </joint>
-            <!-- 0.0 = retract, 0.5 = stop, 1.0 = extend -->
             <joint name="left_linear_actuator_joint">
                 <command_interface name="position">
-                    <param name="min">0.0</param>
+                    <param name="min">-1.0</param>
                     <param name="max">1.0</param>
                 </command_interface>
@@ -112,8 +108,16 @@
             <joint name="right_linear_actuator_joint">
                 <command_interface name="position">
-                    <param name="min">0.0</param>
+                    <param name="min">-1.0</param>
                     <param name="max">1.0</param>
                 </command_interface>
                 <state_interface name="position"/>
+            </joint>
+            <joint name="drum_spin_joint">
+                <command_interface name="velocity">
+                    <param name="min_velocity">-10</param>
+                    <param name="max_velocity">10</param>
+                </command_interface>
+                <state_interface name="position"/>
+                <state_interface name="velocity"/>
             </joint>
         </ros2_control>
