Commit message: jitter fixed

File: qpl_ws/src/qpl_rover/description/rover_core.xacro (robot description, xacro)
@@ -27,5 +27,5 @@
     </collision>
     <xacro:inertial_box mass="10.0" x="${base_x}" y="${base_y}" z="${base_z}">
-      <origin xyz="0 0 ${base_z/2}" rpy="0 0 0"/>
+      <origin xyz="0 0 ${base_z_origin}" rpy="0 0 0"/>
     </xacro:inertial_box>
   </link>
@@ -61,6 +61,6 @@
       <fdir1>1 0 0</fdir1>
       <!-- skid-steer turning: reduce lateral friction -->
-      <mu1>1.0</mu1>
-      <mu2>0.07</mu2>
+      <mu1>1.2</mu1>
+      <mu2>0.05</mu2>
       <!-- optional: allow lateral slip -->
       <slip1>0.0</slip1>

Commit message: imu integration

File: qpl_ws/src/qpl_rover/description/rover_core.xacro (robot description, xacro)
@@ -9,5 +9,6 @@
   <xacro:property name="base_y" value="0.30"/>
   <xacro:property name="base_z" value="0.18"/>
-    <xacro:property name="wheel_r" value="0.08"/>
+  <xacro:property name="wheel_r" value="0.08"/>
+  <!-- base_link is located above the ground by wheel radius + half the base height -->
   <xacro:property name="base_z_origin" value="${wheel_r + base_z/2}"/>
   <xacro:property name="wheel_w" value="0.03"/>
@@ -16,4 +17,7 @@
   <xacro:property name="wheel_y" value="${base_y/2 + wheel_w/2}"/>
   <xacro:property name="wheel_z" value="${wheel_r}"/>
+  <!-- 2D ground-projected base frame -->
+  <link name="base_footprint"/>
+  <!-- Body frame -->
   <link name="base_link">
     <visual>
@@ -30,13 +34,13 @@
     </xacro:inertial_box>
   </link>
+  <!-- base_footprint -> base_link (base_link sits above ground) -->
+  <joint name="base_footprint_joint" type="fixed">
+    <parent link="base_footprint"/>
+    <child link="base_link"/>
+    <origin xyz="0 0 ${base_z_origin}" rpy="0 0 0"/>
+  </joint>
   <gazebo reference="base_link">
     <material>Gazebo/Grey</material>
   </gazebo>
-  <joint name="base_footprint_joint" type="fixed">
-    <parent link="base_link"/>
-    <child link="base_footprint"/>
-    <origin xyz="0 0 0" rpy="0 0 0"/>
-  </joint>
-  <link name="base_footprint"/>
   <!-- WHEELS -->
   <xacro:macro name="wheel_link" params="name">
@@ -56,11 +60,13 @@
       </xacro:inertial_cylinder>
     </link>
+    <gazebo reference="${name}">
+      <material>Gazebo/Red</material>
+    </gazebo>
     <!-- ONE gazebo block per wheel -->
     <gazebo reference="${name}">
-      <material>Gazebo/Red</material>
       <fdir1>1 0 0</fdir1>
       <!-- skid-steer turning: reduce lateral friction -->
-      <mu1>1.2</mu1>
-      <mu2>0.05</mu2>
+      <mu1>1.4</mu1>
+      <mu2>0.07</mu2>
       <!-- optional: allow lateral slip -->
       <slip1>0.0</slip1>

Commit message: Update wheel radius property in rover_core.xacro to 10cm from 8 to match my_controllers.yaml

File: qpl_ws/src/qpl_rover/description/rover_core.xacro (robot description, xacro)
@@ -9,5 +9,5 @@
   <xacro:property name="base_y" value="0.30"/>
   <xacro:property name="base_z" value="0.18"/>
-  <xacro:property name="wheel_r" value="0.08"/>
+  <xacro:property name="wheel_r" value="0.1"/>
   <!-- base_link is located above the ground by wheel radius + half the base height -->
   <xacro:property name="base_z_origin" value="${wheel_r + base_z/2}"/>

Commit message: Update wheel radius from 0.08 to 0.10 to match my_controllers.yaml

File: qpl_ws/src/qpl_rover/description/rover_core.xacro (robot description, xacro)
@@ -9,5 +9,5 @@
   <xacro:property name="base_y" value="0.30"/>
   <xacro:property name="base_z" value="0.18"/>
-  <xacro:property name="wheel_r" value="0.08"/>
+  <xacro:property name="wheel_r" value="0.10"/>
   <!-- base_link is located above the ground by wheel radius + half the base height -->
   <xacro:property name="base_z_origin" value="${wheel_r + base_z/2}"/>

Commit message: twist messages are now floats, bucket is now a cube ontop of rover

File: qpl_ws/src/qpl_rover/description/rover_core.xacro (robot description, xacro)
@@ -119,7 +119,7 @@
   <xacro:property name="drum_mass"   value="1.0"/>
   <!-- Mount at middle of chassis -->
-  <xacro:property name="drum_x" value="${base_x/2 + drum_radius + 0.1}"/>
+  <xacro:property name="drum_x" value="${base_x/2}"/>
   <xacro:property name="drum_y" value="0.0"/>
-  <xacro:property name="drum_z" value="${base_z/2 + drum_radius - 0.1}"/>
+  <xacro:property name="drum_z" value="${base_z/2 + drum_radius +0.25}"/>
   <!-- Drum lift travel: 0 = up (rest), -0.1 = lowered -->
   <xacro:property name="drum_lift_lower" value="-0.1"/>
@@ -141,14 +141,14 @@
   <link name="drum_link">
     <visual>
-      <origin xyz="0 0 0" rpy="${pi/2} 0 0"/>
+      <origin xyz="0 0 0" rpy="0 0 0"/>
       <geometry>
-        <cylinder radius="${drum_radius}" length="${drum_length}"/>
+        <box size="${2*drum_radius} ${drum_length} ${2*drum_radius}"/>
       </geometry>
       <material name="blue"/>
     </visual>
     <collision>
-      <origin xyz="0 0 0" rpy="${pi/2} 0 0"/>
+      <origin xyz="0 0 0" rpy="0 0 0"/>
       <geometry>
-        <cylinder radius="${drum_radius}" length="${drum_length}"/>
+        <box size="${2*drum_radius} ${drum_length} ${2*drum_radius}"/>
       </geometry>
     </collision>

Commit message: initial update of urdf

File: qpl_ws/src/qpl_rover/description/rover_core.xacro (robot description, xacro)
@@ -7,4 +7,8 @@
   <material name="red"><color rgba="0.8 0.1 0.1 1.0"/></material>
   <material name="blue"><color rgba="0.2 0.2 1.0 1.0"/></material>
+  <!-- ========================================================= -->
+  <!-- Robot Dimensions                                          -->
+  <!-- Change these values and the rest of the robot updates      -->
+  <!-- ========================================================= -->
   <!-- Base dimensions -->
   <xacro:property name="base_x" value="0.50"/>
@@ -14,16 +18,28 @@
   <xacro:property name="wheel_r" value="0.15"/>
   <xacro:property name="wheel_w" value="0.03"/>
-  <!-- Frame heights -->
+  <!-- Wheel placement scaling -->
+  <!-- How far from centre the wheels are along the robot length -->
+  <xacro:property name="wheel_x_offset" value="${base_x * 0.36}"/>
+  <!-- Small side clearance between chassis and wheel -->
+  <xacro:property name="wheel_side_clearance" value="0.00"/>
+  <!-- ========================================================= -->
+  <!-- Derived dimensions                                        -->
+  <!-- Do not usually need to edit these                         -->
+  <!-- ========================================================= -->
   <!-- base_footprint is on the ground -->
   <!-- base_link is at chassis centre -->
-  <xacro:property name="base_link_z" value="${wheel_r + base_z/2}"/>
+  <xacro:property name="base_link_z" value="${wheel_r + base_z / 2}"/>
   <!-- Wheel positions relative to base_link -->
-  <xacro:property name="wheel_x_front" value="0.18"/>
-  <xacro:property name="wheel_x_rear"  value="-0.18"/>
-  <xacro:property name="wheel_y" value="${base_y/2 + wheel_w/2}"/>
-  <xacro:property name="wheel_z" value="${-base_z/2}"/>
-  <!-- Ground-projected frame -->
+  <xacro:property name="wheel_x_front" value="${wheel_x_offset}"/>
+  <xacro:property name="wheel_x_rear" value="${-wheel_x_offset}"/>
+  <!-- Wheels sit outside the chassis in Y -->
+  <xacro:property name="wheel_y" value="${base_y / 2 + wheel_w / 2 + wheel_side_clearance}"/>
+  <!-- Wheel centre is level with bottom of chassis -->
+  <!-- This means wheel bottom touches ground because base_link is lifted by wheel_r + base_z/2 -->
+  <xacro:property name="wheel_z" value="${-base_z / 2}"/>
+  <!-- ========================================================= -->
+  <!-- Base frames                                               -->
+  <!-- ========================================================= -->
   <link name="base_footprint"/>
-  <!-- Main body frame -->
   <link name="base_link">
     <visual>
@@ -53,9 +69,12 @@
     <material>Gazebo/Grey</material>
   </gazebo>
-  <!-- Wheel macro -->
+  <!-- ========================================================= -->
+  <!-- Wheel macro                                               -->
+  <!-- ========================================================= -->
   <xacro:macro name="wheel_link" params="name">
     <link name="${name}">
       <visual>
-        <origin xyz="0 0 0" rpy="${pi/2} 0 0"/>
+        <!-- Cylinder is rotated so its axle runs along Y -->
+        <origin xyz="0 0 0" rpy="${pi / 2} 0 0"/>
         <geometry>
           <cylinder radius="${wheel_r}" length="${wheel_w}"/>
@@ -64,7 +83,7 @@
       </visual>
       <collision>
-        <origin xyz="0 0 0" rpy="${pi/2} 0 0"/>
+        <origin xyz="0 0 0" rpy="${pi / 2} 0 0"/>
         <geometry>
-          <cylinder radius="${wheel_r*0.98}" length="${wheel_w*0.95}"/>
+          <cylinder radius="${wheel_r * 0.98}" length="${wheel_w * 0.95}"/>
         </geometry>
       </collision>
@@ -84,10 +103,14 @@
     </gazebo>
   </xacro:macro>
-  <!-- Wheels -->
+  <!-- ========================================================= -->
+  <!-- Wheels                                                    -->
+  <!-- ========================================================= -->
   <xacro:wheel_link name="front_left_wheel"/>
   <xacro:wheel_link name="front_right_wheel"/>
   <xacro:wheel_link name="rear_left_wheel"/>
   <xacro:wheel_link name="rear_right_wheel"/>
-  <!-- Wheel joints -->
+  <!-- ========================================================= -->
+  <!-- Wheel joints                                              -->
+  <!-- ========================================================= -->
   <joint name="front_left_wheel_joint" type="continuous">
     <parent link="base_link"/>

Commit message: added deposition and excivation autonomy

File: qpl_ws/src/qpl_rover/description/rover_core.xacro (robot description, xacro)
@@ -214,7 +214,7 @@
   <xacro:property name="drum_mass"   value="1.0"/>
   <!-- Mount at middle of chassis -->
-  <xacro:property name="drum_x" value="${base_x/2}"/>
+  <xacro:property name="drum_x" value="${base_x/2 - 0.5}"/>
   <xacro:property name="drum_y" value="0.0"/>
-  <xacro:property name="drum_z" value="${base_z/2 + drum_radius +0.25}"/>
+  <xacro:property name="drum_z" value="${base_z/2 + drum_radius + 0.8}"/>
   <!-- Drum lift travel: 0 = up (rest), -0.1 = lowered -->
   <xacro:property name="drum_lift_lower" value="-0.1"/>

Commit message: Update rover_core.xacro

File: qpl_ws/src/qpl_rover/description/rover_core.xacro (robot description, xacro)
@@ -12,5 +12,5 @@
   <!-- Bottom cuboid -->
   <xacro:property name="base_x" value="0.875"/>
-  <xacro:property name="base_y" value="0.599"/>
+  <xacro:property name="base_y" value="0.5806"/>
   <xacro:property name="base_z" value="0.135"/>
   <!-- Top trapezoid section -->

Commit message: Fix sim depth camera topics and rover wheel geometry
- Correct depth camera point cloud topic names in nav_params
  (/depth_camera_*_depth/points) and lower min_obstacle_height to 0.1
- Set rover track from real wheel_separation (0.5836) and raise chassis
  so wheels tuck under the base while keeping ground contact

File: qpl_ws/src/qpl_rover/description/rover_core.xacro (robot description, xacro)
@@ -25,4 +25,11 @@
   <xacro:property name="wheel_r" value="0.15"/>
   <xacro:property name="wheel_w" value="0.15"/>
+  <!-- Real-rover track (centre-to-centre of L/R wheels). Must match -->
+  <!-- diff_cont wheel_separation in config/my_controllers.yaml (0.5836), -->
+  <!-- otherwise sim odometry over-reports yaw and RViz turns faster than Gazebo. -->
+  <xacro:property name="wheel_separation" value="0.5836"/>
+  <!-- Vertical clearance between wheel top and chassis underside so the -->
+  <!-- wheels tuck fully under the base instead of clipping through it. -->
+  <xacro:property name="wheel_base_gap" value="0.01"/>
   <!-- Wheel placement -->
   <xacro:property name="wheel_x_offset" value="${base_x / 2}"/>
@@ -31,11 +38,15 @@
   <!-- Derived values                                            -->
   <!-- ========================================================= -->
-  <!-- Base lift -->
-  <xacro:property name="base_link_z" value="${wheel_r + base_z / 2}"/>
+  <!-- Base lift: raise the chassis so its underside clears the wheel tops -->
+  <!-- (wheel tops sit at 2*wheel_r above ground); wheels still touch ground. -->
+  <xacro:property name="base_link_z" value="${2 * wheel_r + wheel_base_gap + base_z / 2}"/>
   <!-- Wheel positions -->
   <xacro:property name="wheel_x_front" value="${wheel_x_offset}"/>
   <xacro:property name="wheel_x_rear" value="${-wheel_x_offset}"/>
-  <xacro:property name="wheel_y" value="${base_y / 2 + wheel_w / 2 + wheel_side_clearance}"/>
-  <xacro:property name="wheel_z" value="${-base_z / 2}"/>
+  <!-- Track set from the real wheel separation; wheels tuck under the base corners. -->
+  <xacro:property name="wheel_y" value="${wheel_separation / 2}"/>
+  <!-- Hang the wheels below the raised chassis so the wheel centre stays at -->
+  <!-- world z = wheel_r (ground contact): base_link_z + wheel_z = wheel_r. -->
+  <xacro:property name="wheel_z" value="${-(wheel_r + wheel_base_gap + base_z / 2)}"/>
   <!-- Top deck position -->
   <xacro:property name="top_deck_z" value="${base_z / 2 + trap_height + top_z / 2}"/>
