Commit message: Sim wheels: rounded tyre edges
The sim wheel collision was a plain cylinder whose square rim catches on the
terrain mesh while skid-steering. In sim_mode each wheel is now a full-radius
core plus three thinner cylinders per side, stepping down a 4 cm fillet arc
(radius 147 -> 146 -> 142 -> 129 mm). Overall radius and width are unchanged,
so ride height is too. ODE has no filleted shape and mesh-on-mesh contact is
poor, hence the stacked cylinders. The real URDF is unchanged.

Co-Authored-By: Claude Opus 5.5 <noreply@anthropic.com>

File: qpl_ws/src/qpl_rover/description/rover_core.xacro (robot description, xacro)
@@ -333,4 +333,28 @@
   <!-- Wheel macro                                               -->
   <!-- ========================================================= -->
+  <!-- Sim tyre profile: same overall size as the plain collision cylinder below. -->
+  <xacro:property name="tyre_r" value="${wheel_r * 0.98}"/>
+  <xacro:property name="tyre_half_w" value="${wheel_w * 0.95 / 2}"/>
+  <xacro:property name="tyre_fillet" value="0.04"/>
+  <xacro:property name="tyre_slice_w" value="${tyre_fillet / 3}"/>
+  <!-- One pair of edge slices, `index` 1..3 from the core outwards. Each slice takes the
+       arc's radius at its own mid-width. -->
+  <xacro:macro name="tyre_edge_slice" params="index">
+    <xacro:property name="d" value="${(index - 0.5) * tyre_slice_w}"/>
+    <xacro:property name="slice_r" value="${tyre_r - tyre_fillet + (tyre_fillet ** 2 - d ** 2) ** 0.5}"/>
+    <xacro:property name="slice_y" value="${tyre_half_w - tyre_fillet + d}"/>
+    <collision>
+      <origin xyz="0 ${slice_y} 0" rpy="${pi / 2} 0 0"/>
+      <geometry>
+        <cylinder radius="${slice_r}" length="${tyre_slice_w}"/>
+      </geometry>
+    </collision>
+    <collision>
+      <origin xyz="0 ${-slice_y} 0" rpy="${pi / 2} 0 0"/>
+      <geometry>
+        <cylinder radius="${slice_r}" length="${tyre_slice_w}"/>
+      </geometry>
+    </collision>
+  </xacro:macro>
   <xacro:macro name="wheel_link" params="name">
     <link name="${name}">
@@ -342,10 +366,27 @@
         <material name="red"/>
       </visual>
-      <collision>
-        <origin xyz="0 0 0" rpy="${pi / 2} 0 0"/>
-        <geometry>
-          <cylinder radius="${wheel_r * 0.98}" length="${wheel_w * 0.95}"/>
-        </geometry>
-      </collision>
+      <!-- Sim: rounded tyre edges, so the rim doesn't dig into the terrain mesh when
+           skid-steering. ODE has no filleted shape and mesh-on-mesh contact is poor,
+           so the profile is a full-radius core plus three thinner cylinders per side
+           stepping down a tyre_fillet-radius arc. The real URDF keeps the plain cylinder. -->
+      <xacro:if value="$(arg sim_mode)">
+        <collision>
+          <origin xyz="0 0 0" rpy="${pi / 2} 0 0"/>
+          <geometry>
+            <cylinder radius="${tyre_r}" length="${2 * (tyre_half_w - tyre_fillet)}"/>
+          </geometry>
+        </collision>
+        <xacro:tyre_edge_slice index="1"/>
+        <xacro:tyre_edge_slice index="2"/>
+        <xacro:tyre_edge_slice index="3"/>
+      </xacro:if>
+      <xacro:unless value="$(arg sim_mode)">
+        <collision>
+          <origin xyz="0 0 0" rpy="${pi / 2} 0 0"/>
+          <geometry>
+            <cylinder radius="${wheel_r * 0.98}" length="${wheel_w * 0.95}"/>
+          </geometry>
+        </collision>
+      </xacro:unless>
       <xacro:inertial_cylinder mass="0.5" length="${wheel_w}" radius="${wheel_r}">
         <origin xyz="0 0 0" rpy="0 0 0"/>

Commit message: Sim wheels: smooth rounded-rim mesh visual, finer collision profile
The previous commit only changed the collision, so the wheel you see in
Gazebo/RViz was still a sharp-edged cylinder. In sim_mode the wheel visual is
now a tyre mesh with a 4 cm rounded rim between the flat sides and the tread
(description/meshes/wheel.stl, from description/generate_wheel_mesh.py). The
collision follows the same arc in five 8 mm slices per side instead of three.

setup.py installs description/meshes/ (description/* would now pick up the
directory, which setuptools can't copy), and sim.launch.py adds the share
directory to GAZEBO_MODEL_PATH so Gazebo resolves package://qpl_rover meshes.
The real URDF is unchanged.

Co-Authored-By: Claude Opus 5.5 <noreply@anthropic.com>

File: qpl_ws/src/qpl_rover/description/rover_core.xacro (robot description, xacro)
@@ -333,10 +333,11 @@
   <!-- Wheel macro                                               -->
   <!-- ========================================================= -->
-  <!-- Sim tyre profile: same overall size as the plain collision cylinder below. -->
+  <!-- Sim tyre profile: same overall size as the plain collision cylinder below.
+       tyre_fillet must match FILLET in description/generate_wheel_mesh.py (the visual). -->
   <xacro:property name="tyre_r" value="${wheel_r * 0.98}"/>
   <xacro:property name="tyre_half_w" value="${wheel_w * 0.95 / 2}"/>
   <xacro:property name="tyre_fillet" value="0.04"/>
-  <xacro:property name="tyre_slice_w" value="${tyre_fillet / 3}"/>
-  <!-- One pair of edge slices, `index` 1..3 from the core outwards. Each slice takes the
+  <xacro:property name="tyre_slice_w" value="${tyre_fillet / 5}"/>
+  <!-- One pair of edge slices, `index` 1..5 from the core outwards. Each slice takes the
        arc's radius at its own mid-width. -->
   <xacro:macro name="tyre_edge_slice" params="index">
@@ -359,14 +360,26 @@
   <xacro:macro name="wheel_link" params="name">
     <link name="${name}">
-      <visual>
-        <origin xyz="0 0 0" rpy="${pi / 2} 0 0"/>
-        <geometry>
-          <cylinder radius="${wheel_r}" length="${wheel_w}"/>
-        </geometry>
-        <material name="red"/>
-      </visual>
+      <!-- Sim: tyre mesh with a rounded rim (description/generate_wheel_mesh.py), axis along y. -->
+      <xacro:if value="$(arg sim_mode)">
+        <visual>
+          <origin xyz="0 0 0" rpy="0 0 0"/>
+          <geometry>
+            <mesh filename="package://qpl_rover/description/meshes/wheel.stl"/>
+          </geometry>
+          <material name="red"/>
+        </visual>
+      </xacro:if>
+      <xacro:unless value="$(arg sim_mode)">
+        <visual>
+          <origin xyz="0 0 0" rpy="${pi / 2} 0 0"/>
+          <geometry>
+            <cylinder radius="${wheel_r}" length="${wheel_w}"/>
+          </geometry>
+          <material name="red"/>
+        </visual>
+      </xacro:unless>
       <!-- Sim: rounded tyre edges, so the rim doesn't dig into the terrain mesh when
            skid-steering. ODE has no filleted shape and mesh-on-mesh contact is poor,
-           so the profile is a full-radius core plus three thinner cylinders per side
+           so the profile is a full-radius core plus five 8 mm cylinders per side
            stepping down a tyre_fillet-radius arc. The real URDF keeps the plain cylinder. -->
       <xacro:if value="$(arg sim_mode)">
@@ -380,4 +393,6 @@
         <xacro:tyre_edge_slice index="2"/>
         <xacro:tyre_edge_slice index="3"/>
+        <xacro:tyre_edge_slice index="4"/>
+        <xacro:tyre_edge_slice index="5"/>
       </xacro:if>
       <xacro:unless value="$(arg sim_mode)">
